Commit message: right environment generation - try 1

File: ur_workspace_description/urdf/environment_right.urdf.xacro (robot description, xacro)
@@ -3,4 +3,6 @@
   <!-- Materials -->
   <xacro:include filename="$(find ur_workspace_description)/meshes/materials/materials.xacro" />
+  <!-- World Link -->
+  <link name="world"/>
   <!-- Main Table (First Table) -->
   <link name="table_top">

Commit message: right environment generation - try 1

File: ur_workspace_description/urdf/environment_right.urdf.xacro (robot description, xacro)
@@ -49,5 +49,5 @@
     <child link="conveyor_belt"/>
     <!-- Conveyor rotated 90 degrees and positioned between tables -->
-    <origin xyz="-0.77 0 0" rpy="0 0 0"/>
+    <origin xyz="-0.87 0 0" rpy="0 0 0"/>
   </joint>
   <!-- Second Table -->
@@ -139,5 +139,5 @@
     <parent link="table_top"/>
     <child link="safety_barrier_back"/>
-    <origin xyz="0.15 -0.05 0.75" rpy="0 0 0"/>
+    <origin xyz="-0.15 -0.05 0.75" rpy="0 0 0"/>
   </joint>
   <!-- Front Barrier (formerly Left Barrier) -->
@@ -161,5 +161,5 @@
     <parent link="table_top"/>
     <child link="safety_barrier_front"/>
-    <origin xyz="-1.64 -0.05 0.75" rpy="0 0 0"/>
+    <origin xyz="1.64 -0.05 0.75" rpy="0 0 0"/>
   </joint>
   <!-- Top Barrier -->

Commit message: right environment generation - try 1.1

File: ur_workspace_description/urdf/environment_right.urdf.xacro (robot description, xacro)
@@ -132,5 +132,5 @@
       <origin xyz="0 0 0.4" rpy="0 0 1.5708"/>
       <geometry>
-        <box size="-0.05 0.7 0.8"/>
+        <box size="0.05 0.7 0.8"/>
       </geometry>
     </collision>
@@ -154,5 +154,5 @@
       <origin xyz="0 0 0.4" rpy="0 0 1.5708"/>
       <geometry>
-        <box size="-0.05 0.7 0.8"/>
+        <box size="0.05 0.7 0.8"/>
       </geometry>
     </collision>

Commit message: right environment generation - try 1.1

File: ur_workspace_description/urdf/environment_right.urdf.xacro (robot description, xacro)
@@ -139,5 +139,5 @@
     <parent link="table_top"/>
     <child link="safety_barrier_back"/>
-    <origin xyz="-0.15 -0.05 0.75" rpy="0 0 0"/>
+    <origin xyz="0.15 -0.05 0.75" rpy="0 0 0"/>
   </joint>
   <!-- Front Barrier (formerly Left Barrier) -->
@@ -161,5 +161,5 @@
     <parent link="table_top"/>
     <child link="safety_barrier_front"/>
-    <origin xyz="1.64 -0.05 0.75" rpy="0 0 0"/>
+    <origin xyz="-1.64 -0.05 0.75" rpy="0 0 0"/>
   </joint>
   <!-- Top Barrier -->

Commit message: right environment generation - try 1.1

File: ur_workspace_description/urdf/environment_right.urdf.xacro (robot description, xacro)
@@ -139,5 +139,5 @@
     <parent link="table_top"/>
     <child link="safety_barrier_back"/>
-    <origin xyz="0.15 -0.05 0.75" rpy="0 0 0"/>
+    <origin xyz="0.85 -0.05 0.75" rpy="0 0 0"/>
   </joint>
   <!-- Front Barrier (formerly Left Barrier) -->
@@ -161,5 +161,5 @@
     <parent link="table_top"/>
     <child link="safety_barrier_front"/>
-    <origin xyz="-1.64 -0.05 0.75" rpy="0 0 0"/>
+    <origin xyz="-0.85 -0.05 0.75" rpy="0 0 0"/>
   </joint>
   <!-- Top Barrier -->

Commit message: right environment generation - try 1.1

File: ur_workspace_description/urdf/environment_right.urdf.xacro (robot description, xacro)
@@ -161,5 +161,5 @@
     <parent link="table_top"/>
     <child link="safety_barrier_front"/>
-    <origin xyz="-0.85 -0.05 0.75" rpy="0 0 0"/>
+    <origin xyz="-1 -0.05 0.75" rpy="0 0 0"/>
   </joint>
   <!-- Top Barrier -->
