Commit message: Environment approach modification - package 2

File: ur_workspace_description/urdf/environment.urdf.xacro (robot description, xacro)
@@ -10,5 +10,6 @@
       <origin xyz="0 0 0" rpy="0 0 0"/>
       <geometry>
-        <mesh filename="package://ur_workspace_description/meshes/environment/table.stl"/>
+        <!-- Scale down from mm to m -->
+        <mesh filename="package://ur_workspace_description/meshes/environment/table.stl" scale="0.001 0.001 0.001"/>
       </geometry>
       <material name="workspace_light_gray"/>
@@ -31,5 +32,6 @@
       <origin xyz="0 0 0" rpy="0 0 0"/>
       <geometry>
-        <mesh filename="package://ur_workspace_description/meshes/environment/table.stl"/>
+        <!-- Scale down from mm to m -->
+        <mesh filename="package://ur_workspace_description/meshes/environment/table.stl" scale="0.001 0.001 0.001"/>
       </geometry>
       <material name="workspace_light_gray"/>
@@ -52,5 +54,6 @@
       <origin xyz="0 0 0" rpy="0 0 0"/>
       <geometry>
-        <mesh filename="package://ur_workspace_description/meshes/environment/conveyor.stl"/>
+        <!-- Scale down from mm to m -->
+        <mesh filename="package://ur_workspace_description/meshes/environment/conveyor.stl" scale="0.001 0.001 0.001"/>
       </geometry>
       <material name="workspace_dark_gray"/>
@@ -74,5 +77,6 @@
       <origin xyz="0 0 0" rpy="0 0 0"/>
       <geometry>
-        <mesh filename="package://ur_workspace_description/meshes/environment/wide_safety_barrier.stl"/>
+        <!-- Scale down from mm to m -->
+        <mesh filename="package://ur_workspace_description/meshes/environment/wide_safety_barrier.stl" scale="0.001 0.001 0.001"/>
       </geometry>
       <material name="workspace_safety_yellow"/>
@@ -95,5 +99,6 @@
       <origin xyz="0 0 0" rpy="0 0 0"/>
       <geometry>
-        <mesh filename="package://ur_workspace_description/meshes/environment/narrow_safety_barrier.stl"/>
+        <!-- Scale down from mm to m -->
+        <mesh filename="package://ur_workspace_description/meshes/environment/narrow_safety_barrier.stl" scale="0.001 0.001 0.001"/>
       </geometry>
       <material name="workspace_safety_yellow"/>
@@ -116,5 +121,6 @@
       <origin xyz="0 0 0" rpy="0 0 0"/>
       <geometry>
-        <mesh filename="package://ur_workspace_description/meshes/environment/narrow_safety_barrier.stl"/>
+        <!-- Scale down from mm to m -->
+        <mesh filename="package://ur_workspace_description/meshes/environment/narrow_safety_barrier.stl" scale="0.001 0.001 0.001"/>
       </geometry>
       <material name="workspace_safety_yellow"/>
@@ -137,5 +143,6 @@
       <origin xyz="0 0 0" rpy="0 0 0"/>
       <geometry>
-        <mesh filename="package://ur_workspace_description/meshes/environment/wide_safety_barrier.stl"/>
+        <!-- Scale down from mm to m -->
+        <mesh filename="package://ur_workspace_description/meshes/environment/wide_safety_barrier.stl" scale="0.001 0.001 0.001"/>
       </geometry>
       <material name="workspace_safety_yellow"/>
@@ -158,5 +165,6 @@
       <origin xyz="0 0 0" rpy="0 0 0"/>
       <geometry>
-        <mesh filename="package://ur_workspace_description/meshes/environment/top_safety_barrier.stl"/>
+        <!-- Scale down from mm to m -->
+        <mesh filename="package://ur_workspace_description/meshes/environment/top_safety_barrier.stl" scale="0.001 0.001 0.001"/>
       </geometry>
       <material name="workspace_safety_yellow"/>

Commit message: Environment approach modification - package 2.1

File: ur_workspace_description/urdf/environment.urdf.xacro (robot description, xacro)
@@ -25,5 +25,6 @@
     <parent link="world"/>
     <child link="table_top"/>
-    <origin xyz="0 0 0" rpy="0 0 1.5708"/>
+    <!-- Rotated 90 degrees around Z-axis like in reference file -->
+    <origin xyz="0 0 0" rpy="0 0 0"/>
   </joint>
   <!-- Second Table -->
@@ -47,5 +48,6 @@
     <parent link="world"/>
     <child link="table_top_2"/>
-    <origin xyz="1.86 0 0" rpy="0 0 1.5708"/>
+    <!-- Second table positioned on the other side of conveyor with 90-degree rotation -->
+    <origin xyz="1.86 0 0" rpy="0 0 0"/>
   </joint>
   <!-- Conveyor Belt -->
@@ -69,7 +71,8 @@
     <parent link="world"/>
     <child link="conveyor_belt"/>
-    <origin xyz="0.93 0 0" rpy="0 0 1.5708"/>
+    <!-- Conveyor rotated 90 degrees and positioned between tables -->
+    <origin xyz="0.93 0 0" rpy="0 0 0"/>
   </joint>
-  <!-- Safety Barriers -->
+  <!-- Safety Barriers - Adjusted positions for 90-degree rotated tables -->
   <!-- Back Barrier -->
   <link name="safety_barrier_back">
@@ -89,8 +92,9 @@
     </collision>
   </link>
+  <!-- Back barrier positioned at table_length/2 + 0.2 (from reference) -->
   <joint name="table_to_barrier_back" type="fixed">
     <parent link="table_top"/>
     <child link="safety_barrier_back"/>
-    <origin xyz="0 0.45 0.3" rpy="0 0 0"/>
+    <origin xyz="0 0.85 0.3" rpy="0 0 0"/>
   </joint>
   <!-- Right Barrier -->
@@ -111,8 +115,9 @@
     </collision>
   </link>
+  <!-- Right barrier positioned at -table_length/2 + 0.15 (from reference) -->
   <joint name="table_to_barrier_right" type="fixed">
     <parent link="table_top"/>
     <child link="safety_barrier_right"/>
-    <origin xyz="-0.55 0 0.3" rpy="0 0 0"/>
+    <origin xyz="-0.45 0 0.3" rpy="0 0 0"/>
   </joint>
   <!-- Left Barrier -->
@@ -133,8 +138,9 @@
     </collision>
   </link>
+  <!-- Left barrier positioned at table_width/2 + 0.5 (from reference) -->
   <joint name="table_to_barrier_left" type="fixed">
     <parent link="table_top"/>
     <child link="safety_barrier_left"/>
-    <origin xyz="0.55 0 0.3" rpy="0 0 0"/>
+    <origin xyz="0.85 0 0.3" rpy="0 0 0"/>
   </joint>
   <!-- Front Barrier (between table and conveyor) -->
@@ -155,8 +161,9 @@
     </collision>
   </link>
+  <!-- Front barrier positioned at -table_length/2 - conveyor_width + 0.16 (from reference) -->
   <joint name="table_to_barrier_front" type="fixed">
     <parent link="table_top"/>
     <child link="safety_barrier_front"/>
-    <origin xyz="0 -0.45 0.3" rpy="0 0 0"/>
+    <origin xyz="0 -0.84 0.3" rpy="0 0 0"/>
   </joint>
   <!-- Top Barrier -->

Commit message: Environment approach modification - package 2.1

File: ur_workspace_description/urdf/environment.urdf.xacro (robot description, xacro)
@@ -81,5 +81,5 @@
       <geometry>
         <!-- Scale down from mm to m -->
-        <mesh filename="package://ur_workspace_description/meshes/environment/wide_safety_barrier.stl" scale="0.001 0.001 0.001"/>
+        <mesh filename="package://ur_workspace_description/meshes/environment/narrow_safety_barrier.stl" scale="0.001 0.001 0.001"/>
       </geometry>
       <material name="workspace_safety_yellow"/>
@@ -104,5 +104,5 @@
       <geometry>
         <!-- Scale down from mm to m -->
-        <mesh filename="package://ur_workspace_description/meshes/environment/narrow_safety_barrier.stl" scale="0.001 0.001 0.001"/>
+        <mesh filename="package://ur_workspace_description/meshes/environment/wide_safety_barrier.stl" scale="0.001 0.001 0.001"/>
       </geometry>
       <material name="workspace_safety_yellow"/>
@@ -127,5 +127,5 @@
       <geometry>
         <!-- Scale down from mm to m -->
-        <mesh filename="package://ur_workspace_description/meshes/environment/narrow_safety_barrier.stl" scale="0.001 0.001 0.001"/>
+        <mesh filename="package://ur_workspace_description/meshes/environment/wide_safety_barrier.stl" scale="0.001 0.001 0.001"/>
       </geometry>
       <material name="workspace_safety_yellow"/>
@@ -150,5 +150,5 @@
       <geometry>
         <!-- Scale down from mm to m -->
-        <mesh filename="package://ur_workspace_description/meshes/environment/wide_safety_barrier.stl" scale="0.001 0.001 0.001"/>
+        <mesh filename="package://ur_workspace_description/meshes/environment/narrow_safety_barrier.stl" scale="0.001 0.001 0.001"/>
       </geometry>
       <material name="workspace_safety_yellow"/>

Commit message: Environment approach modification - package 2.1

File: ur_workspace_description/urdf/environment.urdf.xacro (robot description, xacro)
@@ -86,5 +86,5 @@
     </visual>
     <collision>
-      <origin xyz="0 0 0.4" rpy="0 0 0"/>
+      <origin xyz="0 0 0.4" rpy="0 0 1.5708"/>
       <geometry>
         <box size="1.2 0.05 0.8"/>
@@ -109,5 +109,5 @@
     </visual>
     <collision>
-      <origin xyz="0 0 0.4" rpy="0 0 0"/>
+      <origin xyz="0 0 0.4" rpy="0 0 1.5708"/>
       <geometry>
         <box size="0.05 0.7 0.8"/>
@@ -132,5 +132,5 @@
     </visual>
     <collision>
-      <origin xyz="0 0 0.4" rpy="0 0 0"/>
+      <origin xyz="0 0 0.4" rpy="0 0 1.5708"/>
       <geometry>
         <box size="0.05 0.7 0.8"/>
@@ -155,5 +155,5 @@
     </visual>
     <collision>
-      <origin xyz="0 0 0.4" rpy="0 0 0"/>
+      <origin xyz="0 0 0.4" rpy="0 0 1.5708"/>
       <geometry>
         <box size="1.2 0.05 0.8"/>

Commit message: Environment approach modification - package 2.2

File: ur_workspace_description/urdf/environment.urdf.xacro (robot description, xacro)
@@ -16,5 +16,5 @@
     </visual>
     <collision>
-      <origin xyz="0 0 0.375" rpy="0 0 0"/>
+      <origin xyz="0 0 0" rpy="0 0 0"/>
       <geometry>
         <box size="1.2 0.7 0.75"/>
@@ -26,5 +26,28 @@
     <child link="table_top"/>
     <!-- Rotated 90 degrees around Z-axis like in reference file -->
-    <origin xyz="0 0 0" rpy="0 0 0"/>
+    <origin xyz="0 0 0.75" rpy="0 0 0"/>
+  </joint>
+  <!-- Conveyor Belt -->
+  <link name="conveyor_belt">
+    <visual>
+      <origin xyz="0 0 0" rpy="0 0 0"/>
+      <geometry>
+        <!-- Scale down from mm to m -->
+        <mesh filename="package://ur_workspace_description/meshes/environment/conveyor.stl" scale="0.001 0.001 0.001"/>
+      </geometry>
+      <material name="workspace_dark_gray"/>
+    </visual>
+    <collision>
+      <origin xyz="0 0 0" rpy="0 0 0"/>
+      <geometry>
+        <box size="2.05 0.8 0.4"/>
+      </geometry>
+    </collision>
+  </link>
+  <joint name="world_to_conveyor" type="fixed">
+    <parent link="world"/>
+    <child link="conveyor_belt"/>
+    <!-- Conveyor rotated 90 degrees and positioned between tables -->
+    <origin xyz="0.83 0.4 0.8" rpy="0 0 0"/>
   </joint>
   <!-- Second Table -->
@@ -39,5 +62,5 @@
     </visual>
     <collision>
-      <origin xyz="0 0 0.375" rpy="0 0 0"/>
+      <origin xyz="0 0 0" rpy="0 0 0"/>
       <geometry>
         <box size="1.2 0.7 0.75"/>
@@ -49,28 +72,5 @@
     <child link="table_top_2"/>
     <!-- Second table positioned on the other side of conveyor with 90-degree rotation -->
-    <origin xyz="1.86 0 0" rpy="0 0 0"/>
-  </joint>
-  <!-- Conveyor Belt -->
-  <link name="conveyor_belt">
-    <visual>
-      <origin xyz="0 0 0" rpy="0 0 0"/>
-      <geometry>
-        <!-- Scale down from mm to m -->
-        <mesh filename="package://ur_workspace_description/meshes/environment/conveyor.stl" scale="0.001 0.001 0.001"/>
-      </geometry>
-      <material name="workspace_dark_gray"/>
-    </visual>
-    <collision>
-      <origin xyz="0 0 0.2" rpy="0 0 0"/>
-      <geometry>
-        <box size="2.05 0.8 0.4"/>
-      </geometry>
-    </collision>
-  </link>
-  <joint name="world_to_conveyor" type="fixed">
-    <parent link="world"/>
-    <child link="conveyor_belt"/>
-    <!-- Conveyor rotated 90 degrees and positioned between tables -->
-    <origin xyz="0.93 0 0" rpy="0 0 0"/>
+    <origin xyz="1.66 0 0.75" rpy="0 0 0"/>
   </joint>
   <!-- Safety Barriers - Adjusted positions for 90-degree rotated tables -->

Commit message: Environment approach modification - package 2.2

File: ur_workspace_description/urdf/environment.urdf.xacro (robot description, xacro)
@@ -26,5 +26,5 @@
     <child link="table_top"/>
     <!-- Rotated 90 degrees around Z-axis like in reference file -->
-    <origin xyz="0 0 0.75" rpy="0 0 0"/>
+    <origin xyz="0 0 0" rpy="0 0 0"/>
   </joint>
   <!-- Conveyor Belt -->
@@ -41,5 +41,5 @@
       <origin xyz="0 0 0" rpy="0 0 0"/>
       <geometry>
-        <box size="2.05 0.8 0.4"/>
+        <box size="2.05 0.8 0"/>
       </geometry>
     </collision>
@@ -49,5 +49,5 @@
     <child link="conveyor_belt"/>
     <!-- Conveyor rotated 90 degrees and positioned between tables -->
-    <origin xyz="0.83 0.4 0.8" rpy="0 0 0"/>
+    <origin xyz="0.83 0 0" rpy="0 0 0"/>
   </joint>
   <!-- Second Table -->
@@ -72,5 +72,5 @@
     <child link="table_top_2"/>
     <!-- Second table positioned on the other side of conveyor with 90-degree rotation -->
-    <origin xyz="1.66 0 0.75" rpy="0 0 0"/>
+    <origin xyz="1.66 0 0" rpy="0 0 0"/>
   </joint>
   <!-- Safety Barriers - Adjusted positions for 90-degree rotated tables -->
@@ -96,5 +96,5 @@
     <parent link="table_top"/>
     <child link="safety_barrier_back"/>
-    <origin xyz="0 0.85 0.3" rpy="0 0 0"/>
+    <origin xyz="0 0.85 0.75" rpy="0 0 0"/>
   </joint>
   <!-- Right Barrier -->
@@ -119,5 +119,5 @@
     <parent link="table_top"/>
     <child link="safety_barrier_right"/>
-    <origin xyz="-0.45 0 0.3" rpy="0 0 0"/>
+    <origin xyz="-0.45 0 0.75" rpy="0 0 0"/>
   </joint>
   <!-- Left Barrier -->
@@ -142,5 +142,5 @@
     <parent link="table_top"/>
     <child link="safety_barrier_left"/>
-    <origin xyz="0.85 0 0.3" rpy="0 0 0"/>
+    <origin xyz="0.85 0 0.75" rpy="0 0 0"/>
   </joint>
   <!-- Front Barrier (between table and conveyor) -->
@@ -165,5 +165,5 @@
     <parent link="table_top"/>
     <child link="safety_barrier_front"/>
-    <origin xyz="0 -0.84 0.3" rpy="0 0 0"/>
+    <origin xyz="0 -0.84 0.75" rpy="0 0 0"/>
   </joint>
   <!-- Top Barrier -->

Commit message: Environment approach modification - package 2.2

File: ur_workspace_description/urdf/environment.urdf.xacro (robot description, xacro)
@@ -26,5 +26,5 @@
     <child link="table_top"/>
     <!-- Rotated 90 degrees around Z-axis like in reference file -->
-    <origin xyz="0 0 0" rpy="0 0 0"/>
+    <origin xyz="0 0.05 0" rpy="0 0 0"/>
   </joint>
   <!-- Conveyor Belt -->
@@ -72,5 +72,5 @@
     <child link="table_top_2"/>
     <!-- Second table positioned on the other side of conveyor with 90-degree rotation -->
-    <origin xyz="1.66 0 0" rpy="0 0 0"/>
+    <origin xyz="1.66 0.05 0" rpy="0 0 0"/>
   </joint>
   <!-- Safety Barriers - Adjusted positions for 90-degree rotated tables -->

Commit message: Environment approach modification - package 2.2

File: ur_workspace_description/urdf/environment.urdf.xacro (robot description, xacro)
@@ -41,5 +41,5 @@
       <origin xyz="0 0 0" rpy="0 0 0"/>
       <geometry>
-        <box size="2.05 0.8 0"/>
+        <box size="2.05 0.85 0"/>
       </geometry>
     </collision>
@@ -49,5 +49,5 @@
     <child link="conveyor_belt"/>
     <!-- Conveyor rotated 90 degrees and positioned between tables -->
-    <origin xyz="0.83 0 0" rpy="0 0 0"/>
+    <origin xyz="0.75 0 0" rpy="0 0 0"/>
   </joint>
   <!-- Second Table -->
@@ -72,5 +72,5 @@
     <child link="table_top_2"/>
     <!-- Second table positioned on the other side of conveyor with 90-degree rotation -->
-    <origin xyz="1.66 0.05 0" rpy="0 0 0"/>
+    <origin xyz="1.65 0.05 0" rpy="0 0 0"/>
   </joint>
   <!-- Safety Barriers - Adjusted positions for 90-degree rotated tables -->
@@ -187,5 +187,5 @@
     <parent link="table_top"/>
     <child link="safety_barrier_top"/>
-    <origin xyz="0 0 1.2" rpy="0 0 0"/>
+    <origin xyz="0 0 2" rpy="0 0 0"/>
   </joint>
 </robot>

Commit message: Environment approach modification - package 2.2

File: ur_workspace_description/urdf/environment.urdf.xacro (robot description, xacro)
@@ -187,5 +187,5 @@
     <parent link="table_top"/>
     <child link="safety_barrier_top"/>
-    <origin xyz="0 0 2" rpy="0 0 0"/>
+    <origin xyz="0 -0.05 2" rpy="0 0 0"/>
   </joint>
 </robot>

Commit message: Environment approach modification - package 2.3

File: ur_workspace_description/urdf/environment.urdf.xacro (robot description, xacro)
@@ -49,5 +49,5 @@
     <child link="conveyor_belt"/>
     <!-- Conveyor rotated 90 degrees and positioned between tables -->
-    <origin xyz="0.75 0 0" rpy="0 0 0"/>
+    <origin xyz="0.8 0 0" rpy="0 0 0"/>
   </joint>
   <!-- Second Table -->
@@ -72,9 +72,9 @@
     <child link="table_top_2"/>
     <!-- Second table positioned on the other side of conveyor with 90-degree rotation -->
-    <origin xyz="1.65 0.05 0" rpy="0 0 0"/>
+    <origin xyz="1.74 0.05 0" rpy="0 0 0"/>
   </joint>
   <!-- Safety Barriers - Adjusted positions for 90-degree rotated tables -->
-  <!-- Back Barrier -->
-  <link name="safety_barrier_back">
+  <!-- Left Barrier (formerly Back Barrier) -->
+  <link name="safety_barrier_left">
     <visual>
       <origin xyz="0 0 0" rpy="0 0 0"/>
@@ -92,12 +92,33 @@
     </collision>
   </link>
-  <!-- Back barrier positioned at table_length/2 + 0.2 (from reference) -->
-  <joint name="table_to_barrier_back" type="fixed">
+  <joint name="table_to_barrier_left" type="fixed">
     <parent link="table_top"/>
-    <child link="safety_barrier_back"/>
-    <origin xyz="0 0.85 0.75" rpy="0 0 0"/>
+    <child link="safety_barrier_left"/>
+    <origin xyz="0 1.55 0.75" rpy="0 0 0"/>
   </joint>
-  <!-- Right Barrier -->
+  <!-- Right Barrier (formerly Front Barrier) -->
   <link name="safety_barrier_right">
+    <visual>
+      <origin xyz="0 0 0" rpy="0 0 0"/>
+      <geometry>
+        <!-- Scale down from mm to m -->
+        <mesh filename="package://ur_workspace_description/meshes/environment/narrow_safety_barrier.stl" scale="0.001 0.001 0.001"/>
+      </geometry>
+      <material name="workspace_safety_yellow"/>
+    </visual>
+    <collision>
+      <origin xyz="0 0 0.4" rpy="0 0 1.5708"/>
+      <geometry>
+        <box size="1.2 0.05 0.8"/>
+      </geometry>
+    </collision>
+  </link>
+  <joint name="table_to_barrier_right" type="fixed">
+    <parent link="table_top"/>
+    <child link="safety_barrier_right"/>
+    <origin xyz="0.25 0 0.75" rpy="0 0 0"/>
+  </joint>
+  <!-- Back Barrier (formerly Right Barrier) -->
+  <link name="safety_barrier_back">
     <visual>
       <origin xyz="0 0 0" rpy="0 0 0"/>
@@ -115,12 +136,11 @@
     </collision>
   </link>
-  <!-- Right barrier positioned at -table_length/2 + 0.15 (from reference) -->
-  <joint name="table_to_barrier_right" type="fixed">
+  <joint name="table_to_barrier_back" type="fixed">
     <parent link="table_top"/>
-    <child link="safety_barrier_right"/>
-    <origin xyz="-0.45 0 0.75" rpy="0 0 0"/>
+    <child link="safety_barrier_back"/>
+    <origin xyz="0 0 0.75" rpy="0 0 0"/>
   </joint>
-  <!-- Left Barrier -->
-  <link name="safety_barrier_left">
+  <!-- Front Barrier (formerly Left Barrier) -->
+  <link name="safety_barrier_front">
     <visual>
       <origin xyz="0 0 0" rpy="0 0 0"/>
@@ -138,32 +158,8 @@
     </collision>
   </link>
-  <!-- Left barrier positioned at table_width/2 + 0.5 (from reference) -->
-  <joint name="table_to_barrier_left" type="fixed">
-    <parent link="table_top"/>
-    <child link="safety_barrier_left"/>
-    <origin xyz="0.85 0 0.75" rpy="0 0 0"/>
-  </joint>
-  <!-- Front Barrier (between table and conveyor) -->
-  <link name="safety_barrier_front">
-    <visual>
-      <origin xyz="0 0 0" rpy="0 0 0"/>
-      <geometry>
-        <!-- Scale down from mm to m -->
-        <mesh filename="package://ur_workspace_description/meshes/environment/narrow_safety_barrier.stl" scale="0.001 0.001 0.001"/>
-      </geometry>
-      <material name="workspace_safety_yellow"/>
-    </visual>
-    <collision>
-      <origin xyz="0 0 0.4" rpy="0 0 1.5708"/>
-      <geometry>
-        <box size="1.2 0.05 0.8"/>
-      </geometry>
-    </collision>
-  </link>
-  <!-- Front barrier positioned at -table_length/2 - conveyor_width + 0.16 (from reference) -->
   <joint name="table_to_barrier_front" type="fixed">
     <parent link="table_top"/>
     <child link="safety_barrier_front"/>
-    <origin xyz="0 -0.84 0.75" rpy="0 0 0"/>
+    <origin xyz="1.2 0 0.75" rpy="0 0 0"/>
   </joint>
   <!-- Top Barrier -->
@@ -187,5 +183,5 @@
     <parent link="table_top"/>
     <child link="safety_barrier_top"/>
-    <origin xyz="0 -0.05 2" rpy="0 0 0"/>
+    <origin xyz="0 -0.05 1.5" rpy="0 0 0"/>
   </joint>
 </robot>

Commit message: Environment approach modification - package 2.3

File: ur_workspace_description/urdf/environment.urdf.xacro (robot description, xacro)
@@ -41,5 +41,5 @@
       <origin xyz="0 0 0" rpy="0 0 0"/>
       <geometry>
-        <box size="2.05 0.85 0"/>
+        <box size="2.05 0.8 0"/>
       </geometry>
     </collision>
@@ -72,5 +72,5 @@
     <child link="table_top_2"/>
     <!-- Second table positioned on the other side of conveyor with 90-degree rotation -->
-    <origin xyz="1.74 0.05 0" rpy="0 0 0"/>
+    <origin xyz="1.64 0.05 0" rpy="0 0 0"/>
   </joint>
   <!-- Safety Barriers - Adjusted positions for 90-degree rotated tables -->
@@ -117,5 +117,5 @@
     <parent link="table_top"/>
     <child link="safety_barrier_right"/>
-    <origin xyz="0.25 0 0.75" rpy="0 0 0"/>
+    <origin xyz="0 0.2 0.75" rpy="0 0 0"/>
   </joint>
   <!-- Back Barrier (formerly Right Barrier) -->
@@ -139,5 +139,5 @@
     <parent link="table_top"/>
     <child link="safety_barrier_back"/>
-    <origin xyz="0 0 0.75" rpy="0 0 0"/>
+    <origin xyz="-0.15 -0.05 0.75" rpy="0 0 0"/>
   </joint>
   <!-- Front Barrier (formerly Left Barrier) -->
@@ -161,5 +161,5 @@
     <parent link="table_top"/>
     <child link="safety_barrier_front"/>
-    <origin xyz="1.2 0 0.75" rpy="0 0 0"/>
+    <origin xyz="1.64 -0.05 0.75" rpy="0 0 0"/>
   </joint>
   <!-- Top Barrier -->

Commit message: Environment approach modification - package 2.3

File: ur_workspace_description/urdf/environment.urdf.xacro (robot description, xacro)
@@ -49,5 +49,5 @@
     <child link="conveyor_belt"/>
     <!-- Conveyor rotated 90 degrees and positioned between tables -->
-    <origin xyz="0.8 0 0" rpy="0 0 0"/>
+    <origin xyz="0.75 0 0" rpy="0 0 0"/>
   </joint>
   <!-- Second Table -->
@@ -183,5 +183,5 @@
     <parent link="table_top"/>
     <child link="safety_barrier_top"/>
-    <origin xyz="0 -0.05 1.5" rpy="0 0 0"/>
+    <origin xyz="0 -0.05 1.75" rpy="0 0 0"/>
   </joint>
 </robot>

Commit message: Environment approach modification - package 2.3

File: ur_workspace_description/urdf/environment.urdf.xacro (robot description, xacro)
@@ -49,5 +49,5 @@
     <child link="conveyor_belt"/>
     <!-- Conveyor rotated 90 degrees and positioned between tables -->
-    <origin xyz="0.75 0 0" rpy="0 0 0"/>
+    <origin xyz="0.77 0 0" rpy="0 0 0"/>
   </joint>
   <!-- Second Table -->
@@ -183,5 +183,5 @@
     <parent link="table_top"/>
     <child link="safety_barrier_top"/>
-    <origin xyz="0 -0.05 1.75" rpy="0 0 0"/>
+    <origin xyz="0 -0.05 1.65" rpy="0 0 0"/>
   </joint>
 </robot>
