Commit message: Robot with environment - fix package 3

File: ur_workspace_description/urdf/environment.urdf.xacro (robot description, xacro)
@@ -3,6 +3,4 @@
   <!-- Materials -->
   <xacro:include filename="$(find ur_workspace_description)/meshes/materials/materials.xacro" />
-  <!-- World Link -->
-  <link name="world"/>
   <!-- Main Table (First Table) -->
   <link name="table_top">
@@ -41,5 +39,5 @@
       <origin xyz="0 0 0" rpy="0 0 0"/>
       <geometry>
-        <box size="2.05 0.8 0.4"/>
+        <box size="2.05 0.8 0"/>
       </geometry>
     </collision>
@@ -48,6 +46,6 @@
     <parent link="world"/>
     <child link="conveyor_belt"/>
-    <!-- Conveyor positioned between tables -->
-    <origin xyz="0.93 0 0" rpy="0 0 1.5708"/>
+    <!-- Conveyor rotated 90 degrees and positioned between tables -->
+    <origin xyz="0.77 0 0" rpy="0 0 0"/>
   </joint>
   <!-- Second Table -->
@@ -71,9 +69,53 @@
     <parent link="world"/>
     <child link="table_top_2"/>
-    <!-- Second table positioned on the other side of conveyor -->
-    <origin xyz="1.86 0.05 0" rpy="0 0 0"/>
+    <!-- Second table positioned on the other side of conveyor with 90-degree rotation -->
+    <origin xyz="1.64 0.05 0" rpy="0 0 0"/>
   </joint>
-  <!-- Safety Barriers -->
-  <!-- Back Barrier -->
+  <!-- Safety Barriers - Adjusted positions for 90-degree rotated tables -->
+  <!-- Left Barrier (formerly Back Barrier) -->
+  <link name="safety_barrier_left">
+    <visual>
+      <origin xyz="0 0 0" rpy="0 0 0"/>
+      <geometry>
+        <!-- Scale down from mm to m -->
+        <mesh filename="package://ur_workspace_description/meshes/environment/narrow_safety_barrier.stl" scale="0.001 0.001 0.001"/>
+      </geometry>
+      <material name="workspace_safety_yellow"/>
+    </visual>
+    <collision>
+      <origin xyz="0 0 0.4" rpy="0 0 1.5708"/>
+      <geometry>
+        <box size="1.2 0.05 0.8"/>
+      </geometry>
+    </collision>
+  </link>
+  <joint name="table_to_barrier_left" type="fixed">
+    <parent link="table_top"/>
+    <child link="safety_barrier_left"/>
+    <origin xyz="0 1.55 0.75" rpy="0 0 0"/>
+  </joint>
+  <!-- Right Barrier (formerly Front Barrier) -->
+  <link name="safety_barrier_right">
+    <visual>
+      <origin xyz="0 0 0" rpy="0 0 0"/>
+      <geometry>
+        <!-- Scale down from mm to m -->
+        <mesh filename="package://ur_workspace_description/meshes/environment/narrow_safety_barrier.stl" scale="0.001 0.001 0.001"/>
+      </geometry>
+      <material name="workspace_safety_yellow"/>
+    </visual>
+    <collision>
+      <origin xyz="0 0 0.4" rpy="0 0 1.5708"/>
+      <geometry>
+        <box size="1.2 0.05 0.8"/>
+      </geometry>
+    </collision>
+  </link>
+  <joint name="table_to_barrier_right" type="fixed">
+    <parent link="table_top"/>
+    <child link="safety_barrier_right"/>
+    <origin xyz="0 0.2 0.75" rpy="0 0 0"/>
+  </joint>
+  <!-- Back Barrier (formerly Right Barrier) -->
   <link name="safety_barrier_back">
     <visual>
@@ -86,7 +128,7 @@
     </visual>
     <collision>
-      <origin xyz="0 0 0.4" rpy="0 0 0"/>
+      <origin xyz="0 0 0.4" rpy="0 0 1.5708"/>
       <geometry>
-        <box size="1.2 0.05 0.8"/>
+        <box size="0.05 0.7 0.8"/>
       </geometry>
     </collision>
@@ -95,7 +137,7 @@
     <parent link="table_top"/>
     <child link="safety_barrier_back"/>
-    <origin xyz="0.0 0.35 0.75" rpy="0 0 0"/>
+    <origin xyz="-0.15 -0.05 0.75" rpy="0 0 0"/>
   </joint>
-  <!-- Front Barrier -->
+  <!-- Front Barrier (formerly Left Barrier) -->
   <link name="safety_barrier_front">
     <visual>
@@ -108,7 +150,7 @@
     </visual>
     <collision>
-      <origin xyz="0 0 0.4" rpy="0 0 0"/>
+      <origin xyz="0 0 0.4" rpy="0 0 1.5708"/>
       <geometry>
-        <box size="1.2 0.05 0.8"/>
+        <box size="0.05 0.7 0.8"/>
       </geometry>
     </collision>
@@ -117,49 +159,5 @@
     <parent link="table_top"/>
     <child link="safety_barrier_front"/>
-    <origin xyz="0.0 -0.35 0.75" rpy="0 0 0"/>
-  </joint>
-  <!-- Left Barrier -->
-  <link name="safety_barrier_left">
-    <visual>
-      <origin xyz="0 0 0" rpy="0 0 0"/>
-      <geometry>
-        <!-- Scale down from mm to m -->
-        <mesh filename="package://ur_workspace_description/meshes/environment/narrow_safety_barrier.stl" scale="0.001 0.001 0.001"/>
-      </geometry>
-      <material name="workspace_safety_yellow"/>
-    </visual>
-    <collision>
-      <origin xyz="0 0 0.4" rpy="0 0 0"/>
-      <geometry>
-        <box size="0.05 0.7 0.8"/>
-      </geometry>
-    </collision>
-  </link>
-  <joint name="table_to_barrier_left" type="fixed">
-    <parent link="table_top"/>
-    <child link="safety_barrier_left"/>
-    <origin xyz="0.6 0.0 0.75" rpy="0 0 0"/>
-  </joint>
-  <!-- Right Barrier -->
-  <link name="safety_barrier_right">
-    <visual>
-      <origin xyz="0 0 0" rpy="0 0 0"/>
-      <geometry>
-        <!-- Scale down from mm to m -->
-        <mesh filename="package://ur_workspace_description/meshes/environment/narrow_safety_barrier.stl" scale="0.001 0.001 0.001"/>
-      </geometry>
-      <material name="workspace_safety_yellow"/>
-    </visual>
-    <collision>
-      <origin xyz="0 0 0.4" rpy="0 0 0"/>
-      <geometry>
-        <box size="0.05 0.7 0.8"/>
-      </geometry>
-    </collision>
-  </link>
-  <joint name="table_to_barrier_right" type="fixed">
-    <parent link="table_top"/>
-    <child link="safety_barrier_right"/>
-    <origin xyz="-0.6 0.0 0.75" rpy="0 0 0"/>
+    <origin xyz="1.64 -0.05 0.75" rpy="0 0 0"/>
   </joint>
   <!-- Top Barrier -->
@@ -176,5 +174,5 @@
       <origin xyz="0 0 0" rpy="0 0 0"/>
       <geometry>
-        <box size="1.2 0.7 0.01"/>
+        <box size="0.7 1.2 0.01"/>
       </geometry>
     </collision>
@@ -183,5 +181,5 @@
     <parent link="table_top"/>
     <child link="safety_barrier_top"/>
-    <origin xyz="0.0 0.0 1.2" rpy="0 0 0"/>
+    <origin xyz="0 -0.05 1.65" rpy="0 0 0"/>
   </joint>
 </robot>

Commit message: barriers replacing

File: ur_workspace_description/urdf/environment.urdf.xacro (robot description, xacro)
@@ -181,5 +181,5 @@
     <parent link="table_top"/>
     <child link="safety_barrier_top"/>
-    <origin xyz="0 -0.05 1.65" rpy="0 0 0"/>
+    <origin xyz="0 -0.05 1.9" rpy="0 0 0"/>
   </joint>
 </robot>

File: ur_workspace_description/urdf/environment_right.urdf.xacro (robot description, xacro)
@@ -161,5 +161,5 @@
     <parent link="table_top"/>
     <child link="safety_barrier_front"/>
-    <origin xyz="-1 -0.05 0.75" rpy="0 0 0"/>
+    <origin xyz="-0.95 -0.05 0.75" rpy="0 0 0"/>
   </joint>
   <!-- Top Barrier -->
@@ -183,5 +183,5 @@
     <parent link="table_top"/>
     <child link="safety_barrier_top"/>
-    <origin xyz="0 -0.05 1.65" rpy="0 0 0"/>
+    <origin xyz="0 -0.05 1.9" rpy="0 0 0"/>
   </joint>
 </robot>
