Commit message: fixing barriers names

File: ur_workspace_description/urdf/Only_environment_for_left_robot.urdf.xacro (robot description, xacro)
@@ -76,4 +76,26 @@
   <!-- Safety Barriers - Adjusted positions for 90-degree rotated tables -->
   <!-- Left Barrier (formerly Back Barrier) -->
+  <link name="safety_barrier_right">
+    <visual>
+      <origin xyz="0 0 0" rpy="0 0 0"/>
+      <geometry>
+        <!-- Scale down from mm to m -->
+        <mesh filename="package://ur_workspace_description/meshes/environment/narrow_safety_barrier.stl" scale="0.001 0.001 0.001"/>
+      </geometry>
+      <material name="workspace_safety_yellow"/>
+    </visual>
+    <collision>
+      <origin xyz="0 0 0.4" rpy="0 0 1.5708"/>
+      <geometry>
+        <box size="-1.2 0.05 0.8"/>
+      </geometry>
+    </collision>
+  </link>
+  <joint name="table_to_barrier_right" type="fixed">
+    <parent link="table_top"/>
+    <child link="safety_barrier_right"/>
+    <origin xyz="0 1.55 0.75" rpy="0 0 0"/>
+  </joint>
+  <!-- Right Barrier (formerly Front Barrier) -->
   <link name="safety_barrier_left">
     <visual>
@@ -95,26 +117,4 @@
     <parent link="table_top"/>
     <child link="safety_barrier_left"/>
-    <origin xyz="0 1.55 0.75" rpy="0 0 0"/>
-  </joint>
-  <!-- Right Barrier (formerly Front Barrier) -->
-  <link name="safety_barrier_right">
-    <visual>
-      <origin xyz="0 0 0" rpy="0 0 0"/>
-      <geometry>
-        <!-- Scale down from mm to m -->
-        <mesh filename="package://ur_workspace_description/meshes/environment/narrow_safety_barrier.stl" scale="0.001 0.001 0.001"/>
-      </geometry>
-      <material name="workspace_safety_yellow"/>
-    </visual>
-    <collision>
-      <origin xyz="0 0 0.4" rpy="0 0 1.5708"/>
-      <geometry>
-        <box size="-1.2 0.05 0.8"/>
-      </geometry>
-    </collision>
-  </link>
-  <joint name="table_to_barrier_right" type="fixed">
-    <parent link="table_top"/>
-    <child link="safety_barrier_right"/>
     <origin xyz="0 0.2 0.75" rpy="0 0 0"/>
   </joint>

File: ur_workspace_description/urdf/left_robot_environment.urdf.xacro (robot description, xacro)
@@ -74,4 +74,26 @@
   <!-- Safety Barriers - Adjusted positions for 90-degree rotated tables -->
   <!-- Left Barrier (formerly Back Barrier) -->
+  <link name="safety_barrier_right">
+    <visual>
+      <origin xyz="0 0 0" rpy="0 0 0"/>
+      <geometry>
+        <!-- Scale down from mm to m -->
+        <mesh filename="package://ur_workspace_description/meshes/environment/narrow_safety_barrier.stl" scale="0.001 0.001 0.001"/>
+      </geometry>
+      <material name="workspace_safety_yellow"/>
+    </visual>
+    <collision>
+      <origin xyz="0 0 0.4" rpy="0 0 1.5708"/>
+      <geometry>
+        <box size="-1.2 0.05 0.8"/>
+      </geometry>
+    </collision>
+  </link>
+  <joint name="table_to_barrier_right" type="fixed">
+    <parent link="table_top"/>
+    <child link="safety_barrier_right"/>
+    <origin xyz="0 1.55 0.75" rpy="0 0 0"/>
+  </joint>
+  <!-- Right Barrier (formerly Front Barrier) -->
   <link name="safety_barrier_left">
     <visual>
@@ -93,26 +115,4 @@
     <parent link="table_top"/>
     <child link="safety_barrier_left"/>
-    <origin xyz="0 1.55 0.75" rpy="0 0 0"/>
-  </joint>
-  <!-- Right Barrier (formerly Front Barrier) -->
-  <link name="safety_barrier_right">
-    <visual>
-      <origin xyz="0 0 0" rpy="0 0 0"/>
-      <geometry>
-        <!-- Scale down from mm to m -->
-        <mesh filename="package://ur_workspace_description/meshes/environment/narrow_safety_barrier.stl" scale="0.001 0.001 0.001"/>
-      </geometry>
-      <material name="workspace_safety_yellow"/>
-    </visual>
-    <collision>
-      <origin xyz="0 0 0.4" rpy="0 0 1.5708"/>
-      <geometry>
-        <box size="-1.2 0.05 0.8"/>
-      </geometry>
-    </collision>
-  </link>
-  <joint name="table_to_barrier_right" type="fixed">
-    <parent link="table_top"/>
-    <child link="safety_barrier_right"/>
     <origin xyz="0 0.2 0.75" rpy="0 0 0"/>
   </joint>

Commit message: Updating Left barrier Position

File: ur_workspace_description/urdf/Only_environment_for_left_robot.urdf.xacro (robot description, xacro)
@@ -117,5 +117,5 @@
     <parent link="table_top"/>
     <child link="safety_barrier_left"/>
-    <origin xyz="0 0.2 0.75" rpy="0 0 0"/>
+    <origin xyz="0 -0.05 0.75" rpy="0 0 0"/>
   </joint>
   <!-- Back Barrier (formerly Right Barrier) -->

File: ur_workspace_description/urdf/left_robot_environment.urdf.xacro (robot description, xacro)
@@ -115,5 +115,5 @@
     <parent link="table_top"/>
     <child link="safety_barrier_left"/>
-    <origin xyz="0 0.2 0.75" rpy="0 0 0"/>
+    <origin xyz="0 -0.05 0.75" rpy="0 0 0"/>
   </joint>
   <!-- Back Barrier (formerly Right Barrier) -->

Commit message: Conveyor belt stl update

File: ur_workspace_description/urdf/Only_environment_for_left_robot.urdf.xacro (robot description, xacro)
@@ -41,5 +41,5 @@
       <origin xyz="0 0 0" rpy="0 0 0"/>
       <geometry>
-        <box size="-2.05 0.8 0"/>
+        <box size="-2.05 0.825 0"/>
       </geometry>
     </collision>

File: ur_workspace_description/urdf/Only_environment_for_right_robot.urdf.xacro (robot description, xacro)
@@ -41,5 +41,5 @@
       <origin xyz="0 0 0" rpy="0 0 0"/>
       <geometry>
-        <box size="2.05 0.8 0"/>
+        <box size="2.05 0.825 0"/>
       </geometry>
     </collision>

File: ur_workspace_description/urdf/left_robot_environment.urdf.xacro (robot description, xacro)
@@ -39,5 +39,5 @@
       <origin xyz="0 0 0" rpy="0 0 0"/>
       <geometry>
-        <box size="-2.05 0.8 0"/>
+        <box size="-2.05 0.825 0"/>
       </geometry>
     </collision>

File: ur_workspace_description/urdf/right_robot_environment.urdf.xacro (robot description, xacro)
@@ -39,5 +39,5 @@
       <origin xyz="0 0 0" rpy="0 0 0"/>
       <geometry>
-        <box size="2.05 0.8 0"/>
+        <box size="2.05 0.825 0"/>
       </geometry>
     </collision>
