Commit message: Environment approach modification

File: ur_workspace_description/meshes/materials/materials.xacro (robot description, xacro)
@@ -16,3 +16,22 @@
     <color rgba="0.1 0.1 0.1 1.0"/>
   </material>
+  <!-- Additional materials from target xacro -->
+  <material name="white">
+    <color rgba="1 1 1 1"/>
+  </material>
+  <material name="brown">
+    <color rgba="0.4 0.2 0 1"/>
+  </material>
+  <material name="red_transparent">
+    <color rgba="1.0 0.0 0.0 0.3"/>
+  </material>
+  <material name="dark_green_rubber">
+    <color rgba="0 0.43 0 1"/>
+  </material>
+  <material name="gray_steel">
+    <color rgba="0.5 0.5 0.5 1"/>
+  </material>
+  <material name="steel">
+    <color rgba="0.5 0.5 0.5 1"/>
+  </material>
 </robot>

File: ur_workspace_description/urdf/environment.urdf.xacro (robot description, xacro)
@@ -5,27 +5,6 @@
   <!-- World Link -->
   <link name="world"/>
-  <!-- Floor -->
-  <link name="floor">
-    <visual>
-      <origin xyz="0 0 -0.05" rpy="0 0 0"/>
-      <geometry>
-        <mesh filename="package://ur_workspace_description/meshes/environment/floor.stl"/>
-      </geometry>
-      <material name="gray"/>
-    </visual>
-    <collision>
-      <origin xyz="0 0 -0.05" rpy="0 0 0"/>
-      <geometry>
-        <box size="4.0 4.0 0.1"/>
-      </geometry>
-    </collision>
-  </link>
-  <joint name="world_to_floor" type="fixed">
-    <parent link="world"/>
-    <child link="floor"/>
-    <origin xyz="0 0 0" rpy="0 0 0"/>
-  </joint>
-  <!-- Main Table -->
-  <link name="main_table">
+  <!-- Main Table (First Table) -->
+  <link name="table_top">
     <visual>
       <origin xyz="0 0 0" rpy="0 0 0"/>
@@ -42,8 +21,29 @@
     </collision>
   </link>
-  <joint name="floor_to_main_table" type="fixed">
-    <parent link="floor"/>
-    <child link="main_table"/>
+  <joint name="world_to_table" type="fixed">
+    <parent link="world"/>
+    <child link="table_top"/>
     <origin xyz="0 0 0" rpy="0 0 1.5708"/>
+  </joint>
+  <!-- Second Table -->
+  <link name="table_top_2">
+    <visual>
+      <origin xyz="0 0 0" rpy="0 0 0"/>
+      <geometry>
+        <mesh filename="package://ur_workspace_description/meshes/environment/table.stl"/>
+      </geometry>
+      <material name="light_gray"/>
+    </visual>
+    <collision>
+      <origin xyz="0 0 0.375" rpy="0 0 0"/>
+      <geometry>
+        <box size="1.2 0.7 0.75"/>
+      </geometry>
+    </collision>
+  </link>
+  <joint name="world_to_table_2" type="fixed">
+    <parent link="world"/>
+    <child link="table_top_2"/>
+    <origin xyz="1.86 0 0" rpy="0 0 1.5708"/>
   </joint>
   <!-- Conveyor Belt -->
@@ -59,19 +59,20 @@
       <origin xyz="0 0 0.2" rpy="0 0 0"/>
       <geometry>
-        <box size="1.5 0.6 0.4"/>
+        <box size="2.05 0.8 0.4"/>
       </geometry>
     </collision>
   </link>
-  <joint name="floor_to_conveyor" type="fixed">
-    <parent link="floor"/>
+  <joint name="world_to_conveyor" type="fixed">
+    <parent link="world"/>
     <child link="conveyor_belt"/>
-    <origin xyz="1.5 0 0" rpy="0 0 0"/>
+    <origin xyz="0.93 0 0" rpy="0 0 1.5708"/>
   </joint>
   <!-- Safety Barriers -->
+  <!-- Back Barrier -->
   <link name="safety_barrier_back">
     <visual>
       <origin xyz="0 0 0" rpy="0 0 0"/>
       <geometry>
-        <mesh filename="package://ur_workspace_description/meshes/environment/barrier.stl"/>
+        <mesh filename="package://ur_workspace_description/meshes/environment/wide_safety_barrier.stl"/>
       </geometry>
       <material name="safety_yellow"/>
@@ -85,8 +86,91 @@
   </link>
   <joint name="table_to_barrier_back" type="fixed">
-    <parent link="main_table"/>
+    <parent link="table_top"/>
     <child link="safety_barrier_back"/>
     <origin xyz="0 0.45 0.3" rpy="0 0 0"/>
   </joint>
-  <!-- Add more barriers as needed -->
+  <!-- Right Barrier -->
+  <link name="safety_barrier_right">
+    <visual>
+      <origin xyz="0 0 0" rpy="0 0 0"/>
+      <geometry>
+        <mesh filename="package://ur_workspace_description/meshes/environment/narrow_safety_barrier.stl"/>
+      </geometry>
+      <material name="safety_yellow"/>
+    </visual>
+    <collision>
+      <origin xyz="0 0 0.4" rpy="0 0 0"/>
+      <geometry>
+        <box size="0.05 0.7 0.8"/>
+      </geometry>
+    </collision>
+  </link>
+  <joint name="table_to_barrier_right" type="fixed">
+    <parent link="table_top"/>
+    <child link="safety_barrier_right"/>
+    <origin xyz="-0.55 0 0.3" rpy="0 0 0"/>
+  </joint>
+  <!-- Left Barrier -->
+  <link name="safety_barrier_left">
+    <visual>
+      <origin xyz="0 0 0" rpy="0 0 0"/>
+      <geometry>
+        <mesh filename="package://ur_workspace_description/meshes/environment/narrow_safety_barrier.stl"/>
+      </geometry>
+      <material name="safety_yellow"/>
+    </visual>
+    <collision>
+      <origin xyz="0 0 0.4" rpy="0 0 0"/>
+      <geometry>
+        <box size="0.05 0.7 0.8"/>
+      </geometry>
+    </collision>
+  </link>
+  <joint name="table_to_barrier_left" type="fixed">
+    <parent link="table_top"/>
+    <child link="safety_barrier_left"/>
+    <origin xyz="0.55 0 0.3" rpy="0 0 0"/>
+  </joint>
+  <!-- Front Barrier (between table and conveyor) -->
+  <link name="safety_barrier_front">
+    <visual>
+      <origin xyz="0 0 0" rpy="0 0 0"/>
+      <geometry>
+        <mesh filename="package://ur_workspace_description/meshes/environment/wide_safety_barrier.stl"/>
+      </geometry>
+      <material name="safety_yellow"/>
+    </visual>
+    <collision>
+      <origin xyz="0 0 0.4" rpy="0 0 0"/>
+      <geometry>
+        <box size="1.2 0.05 0.8"/>
+      </geometry>
+    </collision>
+  </link>
+  <joint name="table_to_barrier_front" type="fixed">
+    <parent link="table_top"/>
+    <child link="safety_barrier_front"/>
+    <origin xyz="0 -0.45 0.3" rpy="0 0 0"/>
+  </joint>
+  <!-- Top Barrier -->
+  <link name="safety_barrier_top">
+    <visual>
+      <origin xyz="0 0 0" rpy="0 0 0"/>
+      <geometry>
+        <mesh filename="package://ur_workspace_description/meshes/environment/top_safety_barrier.stl"/>
+      </geometry>
+      <material name="safety_yellow"/>
+    </visual>
+    <collision>
+      <origin xyz="0 0 0" rpy="0 0 0"/>
+      <geometry>
+        <box size="0.7 1.2 0.01"/>
+      </geometry>
+    </collision>
+  </link>
+  <joint name="table_to_barrier_top" type="fixed">
+    <parent link="table_top"/>
+    <child link="safety_barrier_top"/>
+    <origin xyz="0 0 1.2" rpy="0 0 0"/>
+  </joint>
 </robot>

File: ur_workspace_description/urdf/platform.urdf.xacro (robot description, xacro)
@@ -11,5 +11,5 @@
    <!-- MAIN ROBOT -->
    <xacro:ur_onrobot
-        parent="main_table"
+        parent="table_top"
         robot_ip="$(arg robot_ip)"
         ur_type="$(arg ur_type)"
@@ -25,5 +25,5 @@
         output_recipe_filename="$(find ur_robot_driver)/resources/rtde_output_recipe.txt"
         input_recipe_filename="$(find ur_robot_driver)/resources/rtde_input_recipe.txt">
-        <!-- Robot positioned on table -->
+        <!-- Robot positioned on table - adjusted for new environment -->
         <origin xyz="0.125 -0.225 0.75" rpy="0 0 3.14159"/>
    </xacro:ur_onrobot>

Commit message: Environment approach modification

File: ur_workspace_description/meshes/materials/materials.xacro (robot description, xacro)
@@ -1,36 +1,37 @@
 <?xml version="1.0"?>
 <robot xmlns:xacro="http://www.ros.org/wiki/xacro">
-  <material name="gray">
+  <!-- Use unique prefix for workspace materials to avoid conflicts -->
+  <material name="workspace_gray">
     <color rgba="0.5 0.5 0.5 1.0"/>
   </material>
-  <material name="light_gray">
+  <material name="workspace_light_gray">
     <color rgba="0.8 0.8 0.8 1.0"/>
   </material>
-  <material name="dark_gray">
+  <material name="workspace_dark_gray">
     <color rgba="0.3 0.3 0.3 1.0"/>
   </material>
-  <material name="safety_yellow">
+  <material name="workspace_safety_yellow">
     <color rgba="1.0 1.0 0.0 0.3"/>
   </material>
-  <material name="conveyor_black">
+  <material name="workspace_conveyor_black">
     <color rgba="0.1 0.1 0.1 1.0"/>
   </material>
   <!-- Additional materials from target xacro -->
-  <material name="white">
+  <material name="workspace_white">
     <color rgba="1 1 1 1"/>
   </material>
-  <material name="brown">
+  <material name="workspace_brown">
     <color rgba="0.4 0.2 0 1"/>
   </material>
-  <material name="red_transparent">
+  <material name="workspace_red_transparent">
     <color rgba="1.0 0.0 0.0 0.3"/>
   </material>
-  <material name="dark_green_rubber">
+  <material name="workspace_dark_green_rubber">
     <color rgba="0 0.43 0 1"/>
   </material>
-  <material name="gray_steel">
+  <material name="workspace_gray_steel">
     <color rgba="0.5 0.5 0.5 1"/>
   </material>
-  <material name="steel">
+  <material name="workspace_steel">
     <color rgba="0.5 0.5 0.5 1"/>
   </material>

File: ur_workspace_description/urdf/environment.urdf.xacro (robot description, xacro)
@@ -12,5 +12,5 @@
         <mesh filename="package://ur_workspace_description/meshes/environment/table.stl"/>
       </geometry>
-      <material name="light_gray"/>
+      <material name="workspace_light_gray"/>
     </visual>
     <collision>
@@ -33,5 +33,5 @@
         <mesh filename="package://ur_workspace_description/meshes/environment/table.stl"/>
       </geometry>
-      <material name="light_gray"/>
+      <material name="workspace_light_gray"/>
     </visual>
     <collision>
@@ -54,5 +54,5 @@
         <mesh filename="package://ur_workspace_description/meshes/environment/conveyor.stl"/>
       </geometry>
-      <material name="dark_gray"/>
+      <material name="workspace_dark_gray"/>
     </visual>
     <collision>
@@ -76,5 +76,5 @@
         <mesh filename="package://ur_workspace_description/meshes/environment/wide_safety_barrier.stl"/>
       </geometry>
-      <material name="safety_yellow"/>
+      <material name="workspace_safety_yellow"/>
     </visual>
     <collision>
@@ -97,5 +97,5 @@
         <mesh filename="package://ur_workspace_description/meshes/environment/narrow_safety_barrier.stl"/>
       </geometry>
-      <material name="safety_yellow"/>
+      <material name="workspace_safety_yellow"/>
     </visual>
     <collision>
@@ -118,5 +118,5 @@
         <mesh filename="package://ur_workspace_description/meshes/environment/narrow_safety_barrier.stl"/>
       </geometry>
-      <material name="safety_yellow"/>
+      <material name="workspace_safety_yellow"/>
     </visual>
     <collision>
@@ -139,5 +139,5 @@
         <mesh filename="package://ur_workspace_description/meshes/environment/wide_safety_barrier.stl"/>
       </geometry>
-      <material name="safety_yellow"/>
+      <material name="workspace_safety_yellow"/>
     </visual>
     <collision>
@@ -160,5 +160,5 @@
         <mesh filename="package://ur_workspace_description/meshes/environment/top_safety_barrier.stl"/>
       </geometry>
-      <material name="safety_yellow"/>
+      <material name="workspace_safety_yellow"/>
     </visual>
     <collision>
