Commit message: OnRobot 2FG7 addition - Inclusion package 1

File: ur_onrobot_description/urdf/ur_onrobot_macro.xacro (robot description, xacro)
@@ -26,5 +26,4 @@
             parent="${parent}"
             tf_prefix="${tf_prefix}"
-            use_fake_hardware="${use_fake_hardware}"
             joint_limits_parameters_file="${joint_limits_parameters_file}"
             kinematics_parameters_file="${kinematics_parameters_file}"
@@ -35,5 +34,5 @@
             input_recipe_filename="${input_recipe_filename}"
         >
-            <origin xyz="0 0 0" rpy="0 0 0" />
+            <xacro:insert_block name="origin" />
         </xacro:ur_robot>
         <!--Create the OnRobot model -->

Commit message: rotation fix

File: ur_onrobot_description/urdf/ur_onrobot_macro.xacro (robot description, xacro)
@@ -55,5 +55,5 @@
             <parent link="${tf_prefix}tool0"/>
             <child link="${tf_prefix}onrobot_base_link"/>
-            <origin xyz="0 0 0" rpy="0 0 ${-pi/2}"/>
+            <origin xyz="0 0 0" rpy="0 0 0"/>
         </joint>
         <!-- Include cable connector collision links -->
