Commit message: OnRobot 2FG7 addition - Inclusion package 4

File: ur_onrobot_description/urdf/ur_onrobot.urdf.xacro (robot description, xacro)
@@ -20,5 +20,4 @@
     <xacro:arg name="port" default="502"/>
     <xacro:arg name="device_address" default="65"/>
-    <xacro:arg name="device" default="/tmp/ttyUR"/>
     <xacro:include filename="$(find ur_onrobot_description)/urdf/ur_onrobot_macro.xacro"/>
     <link name="world"/>
@@ -42,5 +41,4 @@
         port="$(arg port)"
         device_address="$(arg device_address)"
-        device="$(arg device)"
         >
         <origin xyz="0 0 1" rpy="0 0 0" />

File: ur_onrobot_description/urdf/ur_onrobot_macro.xacro (robot description, xacro)
@@ -50,5 +50,4 @@
             port="${port}"
             device_address="${device_address}"
-            device="/tmp/ttyUR"
         />
         <!-- Connect the OnRobot to the UR robot -->

File: ur_onrobot_moveit_config/srdf/ur_onrobot_rg.srdf.xacro (robot description, xacro)
@@ -18,4 +18,13 @@
       <joint name="${prefix}finger_width"/>
     </group>
+    <group name="${prefix}${name}_fingers">
+      <joint name="${prefix}finger_joint"/>
+      <joint name="${prefix}left_outer_knuckle_joint"/>
+      <joint name="${prefix}left_inner_knuckle_joint"/>
+      <joint name="${prefix}left_inner_finger_joint"/>
+      <joint name="${prefix}right_outer_knuckle_joint"/>
+      <joint name="${prefix}right_inner_knuckle_joint"/>
+      <joint name="${prefix}right_inner_finger_joint"/>
+    </group>
     <group_state name="closed" group="${prefix}${name}_gripper">
       <joint name="${prefix}finger_width" value="0.0"/>
@@ -33,10 +42,62 @@
     <disable_collisions link1="${prefix}cable_connector_0" link2="${prefix}right_inner_knuckle" reason="Never"/>
     <disable_collisions link1="${prefix}cable_connector_0" link2="${prefix}right_outer_knuckle" reason="Never"/>
-    <!-- Add all your existing RG collision rules here -->
+    <!-- Finger-to-finger collisions -->
     <disable_collisions link1="${prefix}left_inner_finger" link2="${prefix}left_inner_knuckle" reason="Default"/>
     <disable_collisions link1="${prefix}left_inner_finger" link2="${prefix}left_outer_knuckle" reason="Adjacent"/>
     <disable_collisions link1="${prefix}left_inner_finger" link2="${prefix}onrobot_base_link" reason="Never"/>
     <disable_collisions link1="${prefix}left_inner_finger" link2="${prefix}right_inner_finger" reason="Default"/>
-    <!-- Continue with all RG-specific collision rules... -->
+    <disable_collisions link1="${prefix}left_inner_finger" link2="${prefix}right_inner_knuckle" reason="Never"/>
+    <disable_collisions link1="${prefix}left_inner_finger" link2="${prefix}right_outer_knuckle" reason="Never"/>
+    <disable_collisions link1="${prefix}left_inner_finger" link2="${prefix}wrist_1_link" reason="Never"/>
+    <disable_collisions link1="${prefix}left_inner_finger" link2="${prefix}wrist_2_link" reason="Never"/>
+    <disable_collisions link1="${prefix}left_inner_finger" link2="${prefix}wrist_3_link" reason="Never"/>
+    <disable_collisions link1="${prefix}left_inner_knuckle" link2="${prefix}left_outer_knuckle" reason="Default"/>
+    <disable_collisions link1="${prefix}left_inner_knuckle" link2="${prefix}onrobot_base_link" reason="Adjacent"/>
+    <disable_collisions link1="${prefix}left_inner_knuckle" link2="${prefix}right_inner_finger" reason="Never"/>
+    <disable_collisions link1="${prefix}left_inner_knuckle" link2="${prefix}right_inner_knuckle" reason="Never"/>
+    <disable_collisions link1="${prefix}left_inner_knuckle" link2="${prefix}right_outer_knuckle" reason="Never"/>
+    <disable_collisions link1="${prefix}left_inner_knuckle" link2="${prefix}wrist_1_link" reason="Never"/>
+    <disable_collisions link1="${prefix}left_inner_knuckle" link2="${prefix}wrist_2_link" reason="Never"/>
+    <disable_collisions link1="${prefix}left_inner_knuckle" link2="${prefix}wrist_3_link" reason="Never"/>
+    <disable_collisions link1="${prefix}left_outer_knuckle" link2="${prefix}onrobot_base_link" reason="Adjacent"/>
+    <disable_collisions link1="${prefix}left_outer_knuckle" link2="${prefix}right_inner_finger" reason="Never"/>
+    <disable_collisions link1="${prefix}left_outer_knuckle" link2="${prefix}right_inner_knuckle" reason="Never"/>
+    <disable_collisions link1="${prefix}left_outer_knuckle" link2="${prefix}right_outer_knuckle" reason="Never"/>
+    <disable_collisions link1="${prefix}left_outer_knuckle" link2="${prefix}wrist_1_link" reason="Never"/>
+    <disable_collisions link1="${prefix}left_outer_knuckle" link2="${prefix}wrist_2_link" reason="Never"/>
+    <disable_collisions link1="${prefix}left_outer_knuckle" link2="${prefix}wrist_3_link" reason="Never"/>
+    <disable_collisions link1="${prefix}onrobot_base_link" link2="${prefix}right_inner_finger" reason="Never"/>
+    <disable_collisions link1="${prefix}onrobot_base_link" link2="${prefix}right_inner_knuckle" reason="Adjacent"/>
+    <disable_collisions link1="${prefix}onrobot_base_link" link2="${prefix}right_outer_knuckle" reason="Adjacent"/>
+    <disable_collisions link1="${prefix}right_inner_finger" link2="${prefix}right_inner_knuckle" reason="Default"/>
+    <disable_collisions link1="${prefix}right_inner_finger" link2="${prefix}right_outer_knuckle" reason="Adjacent"/>
+    <disable_collisions link1="${prefix}right_inner_finger" link2="${prefix}wrist_1_link" reason="Never"/>
+    <disable_collisions link1="${prefix}right_inner_finger" link2="${prefix}wrist_2_link" reason="Never"/>
+    <disable_collisions link1="${prefix}right_inner_finger" link2="${prefix}wrist_3_link" reason="Never"/>
+    <disable_collisions link1="${prefix}right_inner_knuckle" link2="${prefix}right_outer_knuckle" reason="Default"/>
+    <disable_collisions link1="${prefix}right_inner_knuckle" link2="${prefix}wrist_1_link" reason="Never"/>
+    <disable_collisions link1="${prefix}right_inner_knuckle" link2="${prefix}wrist_2_link" reason="Never"/>
+    <disable_collisions link1="${prefix}right_inner_knuckle" link2="${prefix}wrist_3_link" reason="Never"/>
+    <disable_collisions link1="${prefix}right_outer_knuckle" link2="${prefix}wrist_1_link" reason="Never"/>
+    <disable_collisions link1="${prefix}right_outer_knuckle" link2="${prefix}wrist_2_link" reason="Never"/>
+    <disable_collisions link1="${prefix}right_outer_knuckle" link2="${prefix}wrist_3_link" reason="Never"/>
+    <!-- Finger tip collisions -->
+    <disable_collisions link1="${prefix}left_finger_tip" link2="${prefix}right_finger_tip" reason="Default"/>
+    <disable_collisions link1="${prefix}left_finger_tip" link2="${prefix}onrobot_base_link" reason="Never"/>
+    <disable_collisions link1="${prefix}left_finger_tip" link2="${prefix}left_inner_finger" reason="Adjacent"/>
+    <disable_collisions link1="${prefix}left_finger_tip" link2="${prefix}right_inner_finger" reason="Default"/>
+    <disable_collisions link1="${prefix}right_finger_tip" link2="${prefix}onrobot_base_link" reason="Never"/>
+    <disable_collisions link1="${prefix}right_finger_tip" link2="${prefix}right_inner_finger" reason="Adjacent"/>
+    <!-- Cable connector collisions with robot arm -->
+    <disable_collisions link1="${prefix}cable_connector_0" link2="${prefix}wrist_1_link" reason="Never"/>
+    <disable_collisions link1="${prefix}cable_connector_0" link2="${prefix}wrist_2_link" reason="Never"/>
+    <disable_collisions link1="${prefix}cable_connector_0" link2="${prefix}wrist_3_link" reason="Default"/>
+    <disable_collisions link1="${prefix}cable_connector_1" link2="${prefix}wrist_1_link" reason="Never"/>
+    <disable_collisions link1="${prefix}cable_connector_1" link2="${prefix}wrist_2_link" reason="Default"/>
+    <disable_collisions link1="${prefix}cable_connector_1" link2="${prefix}wrist_3_link" reason="Default"/>
+    <!-- Gripper base to robot arm collisions -->
+    <disable_collisions link1="${prefix}onrobot_base_link" link2="${prefix}wrist_1_link" reason="Never"/>
+    <disable_collisions link1="${prefix}onrobot_base_link" link2="${prefix}wrist_2_link" reason="Never"/>
+    <disable_collisions link1="${prefix}onrobot_base_link" link2="${prefix}wrist_3_link" reason="Adjacent"/>
   </xacro:macro>
 </robot>

File: ur_workspace_description/urdf/platform.urdf.xacro (robot description, xacro)
@@ -14,5 +14,4 @@
    <xacro:arg name="port" default="502"/>
    <xacro:arg name="device_address" default="65"/>
-   <xacro:arg name="device" default="/tmp/ttyUR"/>
    <!-- MAIN ROBOT -->
    <xacro:ur_onrobot
@@ -35,5 +34,5 @@
         port="$(arg port)"
         device_address="$(arg device_address)"
-        device="$(arg device)">
+        >
         <!-- Robot positioned on table - adjusted for new environment -->
         <origin xyz="0.125 -0.225 0.75" rpy="0 0 3.14159"/>

Commit message: repositioning robot in RVIZ

File: ur_onrobot_description/urdf/ur_onrobot.urdf.xacro (robot description, xacro)
@@ -42,5 +42,5 @@
         device_address="$(arg device_address)"
         >
-        <origin xyz="0 0 1" rpy="0 0 0" />
+        <origin xyz="0 0 0" rpy="0 0 0" />
     </xacro:ur_onrobot>
 </robot>

Commit message: description package fix

File: ur_onrobot_description/urdf/ur_onrobot.urdf.xacro (robot description, xacro)
@@ -2,5 +2,5 @@
 <robot name="ur_onrobot" xmlns:xacro="http://ros.org/wiki/xacro">
     <!-- Arguments -->
-    <xacro:arg name="robot_ip" default="192.168.1.101"/>
+    <xacro:arg name="robot_ip" default="192.168.1.105"/>
     <xacro:arg name="ur_type" default="ur5e"/>
     <xacro:arg name="onrobot_type" default="2fg7"/>
@@ -20,5 +20,4 @@
     <xacro:arg name="port" default="502"/>
     <xacro:arg name="device_address" default="65"/>
-    <xacro:arg name="device" default="/tmp/ttyUR"/>
     <xacro:include filename="$(find ur_onrobot_description)/urdf/ur_onrobot_macro.xacro"/>
     <link name="world"/>
@@ -42,7 +41,6 @@
         port="$(arg port)"
         device_address="$(arg device_address)"
-        device="$(arg device)"
         >
-        <origin xyz="0 0 0" rpy="0 0 0" />
+        <origin xyz="0 0 1" rpy="0 0 0" />
     </xacro:ur_onrobot>
 </robot>

File: ur_onrobot_description/urdf/ur_onrobot_macro.xacro (robot description, xacro)
@@ -23,5 +23,4 @@
         port:=502
         device_address:=65
-        device:=/tmp/ttyUR
         ">
         <!-- Create the UR robot -->
@@ -51,5 +50,4 @@
             port="${port}"
             device_address="${device_address}"
-            device="${device}"
         />
         <!-- Connect the OnRobot to the UR robot -->

Commit message: back to basics

File: ur_onrobot_description/urdf/ur_onrobot.urdf.xacro (robot description, xacro)
@@ -2,5 +2,5 @@
 <robot name="ur_onrobot" xmlns:xacro="http://ros.org/wiki/xacro">
     <!-- Arguments -->
-    <xacro:arg name="robot_ip" default="192.168.1.105"/>
+    <xacro:arg name="robot_ip" default="192.168.56.101"/>
     <xacro:arg name="ur_type" default="ur5e"/>
     <xacro:arg name="onrobot_type" default="2fg7"/>
@@ -15,9 +15,4 @@
     <xacro:arg name="input_recipe_filename" default="$(find ur_robot_driver)/resources/rtde_input_recipe.txt"/>
     <xacro:arg name="output_recipe_filename" default="$(find ur_robot_driver)/resources/rtde_output_recipe.txt"/>
-    <!-- MODBUS parameters -->
-    <xacro:arg name="connection_type" default="tcp"/>
-    <xacro:arg name="ip_address" default="192.168.1.1"/>
-    <xacro:arg name="port" default="502"/>
-    <xacro:arg name="device_address" default="65"/>
     <xacro:include filename="$(find ur_onrobot_description)/urdf/ur_onrobot_macro.xacro"/>
     <link name="world"/>
@@ -37,8 +32,4 @@
         output_recipe_filename="$(arg output_recipe_filename)"
         input_recipe_filename="$(arg input_recipe_filename)"
-        connection_type="$(arg connection_type)"
-        ip_address="$(arg ip_address)"
-        port="$(arg port)"
-        device_address="$(arg device_address)"
         >
         <origin xyz="0 0 1" rpy="0 0 0" />

File: ur_onrobot_description/urdf/ur_onrobot_macro.xacro (robot description, xacro)
@@ -19,10 +19,6 @@
         output_recipe_filename
         input_recipe_filename
-        connection_type:=tcp
-        ip_address:=192.168.1.1
-        port:=502
-        device_address:=65
         ">
-        <!-- Create the UR robot -->
+        <!-- Create the UR robot-->
         <xacro:ur_robot
             robot_ip="${robot_ip}"
@@ -39,15 +35,11 @@
             input_recipe_filename="${input_recipe_filename}"
         >
-            <xacro:insert_block name="origin" />
+            <origin xyz="0 0 0" rpy="0 0 0" />
         </xacro:ur_robot>
-        <!--Create the OnRobot model with ALL parameters -->
+        <!--Create the OnRobot model -->
         <xacro:onrobot
             onrobot_type="${onrobot_type}"
             prefix="${tf_prefix}"
             use_fake_hardware="${use_fake_hardware}"
-            connection_type="${connection_type}"
-            ip_address="${ip_address}"
-            port="${port}"
-            device_address="${device_address}"
         />
         <!-- Connect the OnRobot to the UR robot -->

Commit message: enrique's working version

File: ur_onrobot_description/urdf/ur_onrobot.urdf.xacro (robot description, xacro)
@@ -2,5 +2,5 @@
 <robot name="ur_onrobot" xmlns:xacro="http://ros.org/wiki/xacro">
     <!-- Arguments -->
-    <xacro:arg name="robot_ip" default="192.168.56.101"/>
+    <xacro:arg name="robot_ip" default="192.168.1.105"/>
     <xacro:arg name="ur_type" default="ur5e"/>
     <xacro:arg name="onrobot_type" default="2fg7"/>
@@ -15,4 +15,9 @@
     <xacro:arg name="input_recipe_filename" default="$(find ur_robot_driver)/resources/rtde_input_recipe.txt"/>
     <xacro:arg name="output_recipe_filename" default="$(find ur_robot_driver)/resources/rtde_output_recipe.txt"/>
+    <!-- MODBUS parameters -->
+    <xacro:arg name="connection_type" default="tcp"/>
+    <xacro:arg name="ip_address" default="192.168.1.1"/>
+    <xacro:arg name="port" default="502"/>
+    <xacro:arg name="device_address" default="65"/>
     <xacro:include filename="$(find ur_onrobot_description)/urdf/ur_onrobot_macro.xacro"/>
     <link name="world"/>
@@ -32,4 +37,8 @@
         output_recipe_filename="$(arg output_recipe_filename)"
         input_recipe_filename="$(arg input_recipe_filename)"
+        connection_type="$(arg connection_type)"
+        ip_address="$(arg ip_address)"
+        port="$(arg port)"
+        device_address="$(arg device_address)"
         >
         <origin xyz="0 0 1" rpy="0 0 0" />

File: ur_onrobot_description/urdf/ur_onrobot_macro.xacro (robot description, xacro)
@@ -19,6 +19,10 @@
         output_recipe_filename
         input_recipe_filename
+        connection_type:=tcp
+        ip_address:=192.168.1.1
+        port:=502
+        device_address:=65
         ">
-        <!-- Create the UR robot-->
+        <!-- Create the UR robot -->
         <xacro:ur_robot
             robot_ip="${robot_ip}"
@@ -35,11 +39,15 @@
             input_recipe_filename="${input_recipe_filename}"
         >
-            <origin xyz="0 0 0" rpy="0 0 0" />
+            <xacro:insert_block name="origin" />
         </xacro:ur_robot>
-        <!--Create the OnRobot model -->
+        <!--Create the OnRobot model with ALL parameters -->
         <xacro:onrobot
             onrobot_type="${onrobot_type}"
             prefix="${tf_prefix}"
             use_fake_hardware="${use_fake_hardware}"
+            connection_type="${connection_type}"
+            ip_address="${ip_address}"
+            port="${port}"
+            device_address="${device_address}"
         />
         <!-- Connect the OnRobot to the UR robot -->
