Commit message: Robot with environment - fix package 1

File: ur_onrobot_control/urdf/robot_with_environment.urdf.xacro (robot description, xacro)
@@ -1,5 +1,5 @@
 <?xml version='1.0' encoding='utf-8'?>
-<robot xmlns:xacro="http://www.ros.org/wiki/xacro" name="platform">
-   <!-- Include the environment -->
+<robot xmlns:xacro="http://www.ros.org/wiki/xacro" name="ur_onrobot_with_environment">
+   <!-- Include the environment (keeping environment.urdf.xacro exactly as is) -->
    <xacro:include filename="$(find ur_workspace_description)/urdf/environment.urdf.xacro"/>
    <!-- Include the complete UR+OnRobot description -->
@@ -9,4 +9,5 @@
    <xacro:arg name="robot_ip" default="192.168.1.101" />
    <xacro:arg name="use_fake_hardware" default="true" />
+   <xacro:arg name="tf_prefix" default=""/>
    <!-- MODBUS parameters for 2FG7 -->
    <xacro:arg name="connection_type" default="tcp"/>
@@ -14,5 +15,5 @@
    <xacro:arg name="port" default="502"/>
    <xacro:arg name="device_address" default="65"/>
-   <!-- MAIN ROBOT -->
+   <!-- MAIN ROBOT - Attached to the table in the environment -->
    <xacro:ur_onrobot
         parent="table_top"
@@ -20,5 +21,5 @@
         ur_type="$(arg ur_type)"
         onrobot_type="$(arg onrobot_type)"
-        tf_prefix=""
+        tf_prefix="$(arg tf_prefix)"
         use_fake_hardware="$(arg use_fake_hardware)"
         cable_connector="true"
@@ -35,6 +36,6 @@
         device_address="$(arg device_address)"
         >
-        <!-- Robot positioned on table - adjusted for new environment -->
-        <origin xyz="0.125 -0.225 0.75" rpy="0 0 3.14159"/>
+        <!-- Robot positioned on table - centered on first table -->
+        <origin xyz="0.6 0.35 0.75" rpy="0 0 0"/>
    </xacro:ur_onrobot>
 </robot>

Commit message: Robot with environment - fix package 1

File: ur_onrobot_control/urdf/robot_with_environment.urdf.xacro (robot description, xacro)
@@ -1,7 +1,9 @@
 <?xml version='1.0' encoding='utf-8'?>
 <robot xmlns:xacro="http://www.ros.org/wiki/xacro" name="ur_onrobot_with_environment">
-   <!-- Include the environment (keeping environment.urdf.xacro exactly as is) -->
+   <!-- World Link -->
+   <link name="world"/>
+   <!-- Include environment components individually to avoid material conflicts -->
    <xacro:include filename="$(find ur_workspace_description)/urdf/environment.urdf.xacro"/>
-   <!-- Include the complete UR+OnRobot description -->
+   <!-- Create a separate robot description without material conflicts -->
    <xacro:include filename="$(find ur_onrobot_description)/urdf/ur_onrobot.urdf.xacro"/>
    <xacro:arg name="ur_type" default="ur5e"/>
@@ -23,4 +25,5 @@
         tf_prefix="$(arg tf_prefix)"
         use_fake_hardware="$(arg use_fake_hardware)"
+        name="ur_robot"
         cable_connector="true"
         joint_limits_parameters_file="$(find ur_description)/config/$(arg ur_type)/joint_limits.yaml"

Commit message: Robot with environment - fix package 2

File: ur_onrobot_control/urdf/robot_with_environment.urdf.xacro (robot description, xacro)
@@ -3,8 +3,8 @@
    <!-- World Link -->
    <link name="world"/>
-   <!-- Include environment components individually to avoid material conflicts -->
+   <!-- Include environment components -->
    <xacro:include filename="$(find ur_workspace_description)/urdf/environment.urdf.xacro"/>
-   <!-- Create a separate robot description without material conflicts -->
-   <xacro:include filename="$(find ur_onrobot_description)/urdf/ur_onrobot.urdf.xacro"/>
+   <!-- Create robot description -->
+   <xacro:include filename="$(find ur_onrobot_description)/urdf/ur_onrobot_macro.xacro"/>
    <xacro:arg name="ur_type" default="ur5e"/>
    <xacro:arg name="onrobot_type" default="2fg7"/>
@@ -17,5 +17,13 @@
    <xacro:arg name="port" default="502"/>
    <xacro:arg name="device_address" default="65"/>
-   <!-- MAIN ROBOT - Attached to the table in the environment -->
+   <!-- Joint limits and other UR parameters -->
+   <xacro:arg name="joint_limits_parameters_file" default="$(find ur_description)/config/$(arg ur_type)/joint_limits.yaml"/>
+   <xacro:arg name="kinematics_parameters_file" default="$(find ur_description)/config/$(arg ur_type)/default_kinematics.yaml"/>
+   <xacro:arg name="physical_parameters_file" default="$(find ur_description)/config/$(arg ur_type)/physical_parameters.yaml"/>
+   <xacro:arg name="visual_parameters_file" default="$(find ur_description)/config/$(arg ur_type)/visual_parameters.yaml"/>
+   <xacro:arg name="script_filename" default="$(find ur_robot_driver)/resources/ros_control.urscript"/>
+   <xacro:arg name="output_recipe_filename" default="$(find ur_robot_driver)/resources/rtde_output_recipe.txt"/>
+   <xacro:arg name="input_recipe_filename" default="$(find ur_robot_driver)/resources/rtde_input_recipe.txt"/>
+   <!-- MAIN ROBOT - Attached to the first table in the environment -->
    <xacro:ur_onrobot
         parent="table_top"
@@ -25,20 +33,18 @@
         tf_prefix="$(arg tf_prefix)"
         use_fake_hardware="$(arg use_fake_hardware)"
-        name="ur_robot"
-        cable_connector="true"
-        joint_limits_parameters_file="$(find ur_description)/config/$(arg ur_type)/joint_limits.yaml"
-        kinematics_parameters_file="$(find ur_description)/config/$(arg ur_type)/default_kinematics.yaml"
-        physical_parameters_file="$(find ur_description)/config/$(arg ur_type)/physical_parameters.yaml"
-        visual_parameters_file="$(find ur_description)/config/$(arg ur_type)/visual_parameters.yaml"
-        script_filename="$(find ur_robot_driver)/resources/ros_control.urscript"
-        output_recipe_filename="$(find ur_robot_driver)/resources/rtde_output_recipe.txt"
-        input_recipe_filename="$(find ur_robot_driver)/resources/rtde_input_recipe.txt"
+        joint_limits_parameters_file="$(arg joint_limits_parameters_file)"
+        kinematics_parameters_file="$(arg kinematics_parameters_file)"
+        physical_parameters_file="$(arg physical_parameters_file)"
+        visual_parameters_file="$(arg visual_parameters_file)"
+        script_filename="$(arg script_filename)"
+        output_recipe_filename="$(arg output_recipe_filename)"
+        input_recipe_filename="$(arg input_recipe_filename)"
         connection_type="$(arg connection_type)"
         ip_address="$(arg ip_address)"
         port="$(arg port)"
         device_address="$(arg device_address)"
-        >
-        <!-- Robot positioned on table - centered on first table -->
-        <origin xyz="0.6 0.35 0.75" rpy="0 0 0"/>
+        cable_connector="true">
+        <!-- Robot positioned on table - adjust as needed -->
+        <origin xyz="0.0 0.0 0.75" rpy="0 0 0"/>
    </xacro:ur_onrobot>
 </robot>

File: ur_workspace_description/urdf/environment.urdf_bk.xacro (robot description, xacro)
@@ -41,5 +41,5 @@
       <origin xyz="0 0 0" rpy="0 0 0"/>
       <geometry>
-        <box size="2.05 0.8 0.4"/>
+        <box size="2.05 0.8 0"/>
       </geometry>
     </collision>
@@ -48,6 +48,6 @@
     <parent link="world"/>
     <child link="conveyor_belt"/>
-    <!-- Conveyor positioned between tables -->
-    <origin xyz="0.93 0 0" rpy="0 0 1.5708"/>
+    <!-- Conveyor rotated 90 degrees and positioned between tables -->
+    <origin xyz="0.77 0 0" rpy="0 0 0"/>
   </joint>
   <!-- Second Table -->
@@ -71,9 +71,53 @@
     <parent link="world"/>
     <child link="table_top_2"/>
-    <!-- Second table positioned on the other side of conveyor -->
-    <origin xyz="1.86 0.05 0" rpy="0 0 0"/>
+    <!-- Second table positioned on the other side of conveyor with 90-degree rotation -->
+    <origin xyz="1.64 0.05 0" rpy="0 0 0"/>
   </joint>
-  <!-- Safety Barriers -->
-  <!-- Back Barrier -->
+  <!-- Safety Barriers - Adjusted positions for 90-degree rotated tables -->
+  <!-- Left Barrier (formerly Back Barrier) -->
+  <link name="safety_barrier_left">
+    <visual>
+      <origin xyz="0 0 0" rpy="0 0 0"/>
+      <geometry>
+        <!-- Scale down from mm to m -->
+        <mesh filename="package://ur_workspace_description/meshes/environment/narrow_safety_barrier.stl" scale="0.001 0.001 0.001"/>
+      </geometry>
+      <material name="workspace_safety_yellow"/>
+    </visual>
+    <collision>
+      <origin xyz="0 0 0.4" rpy="0 0 1.5708"/>
+      <geometry>
+        <box size="1.2 0.05 0.8"/>
+      </geometry>
+    </collision>
+  </link>
+  <joint name="table_to_barrier_left" type="fixed">
+    <parent link="table_top"/>
+    <child link="safety_barrier_left"/>
+    <origin xyz="0 1.55 0.75" rpy="0 0 0"/>
+  </joint>
+  <!-- Right Barrier (formerly Front Barrier) -->
+  <link name="safety_barrier_right">
+    <visual>
+      <origin xyz="0 0 0" rpy="0 0 0"/>
+      <geometry>
+        <!-- Scale down from mm to m -->
+        <mesh filename="package://ur_workspace_description/meshes/environment/narrow_safety_barrier.stl" scale="0.001 0.001 0.001"/>
+      </geometry>
+      <material name="workspace_safety_yellow"/>
+    </visual>
+    <collision>
+      <origin xyz="0 0 0.4" rpy="0 0 1.5708"/>
+      <geometry>
+        <box size="1.2 0.05 0.8"/>
+      </geometry>
+    </collision>
+  </link>
+  <joint name="table_to_barrier_right" type="fixed">
+    <parent link="table_top"/>
+    <child link="safety_barrier_right"/>
+    <origin xyz="0 0.2 0.75" rpy="0 0 0"/>
+  </joint>
+  <!-- Back Barrier (formerly Right Barrier) -->
   <link name="safety_barrier_back">
     <visual>
@@ -86,7 +130,7 @@
     </visual>
     <collision>
-      <origin xyz="0 0 0.4" rpy="0 0 0"/>
+      <origin xyz="0 0 0.4" rpy="0 0 1.5708"/>
       <geometry>
-        <box size="1.2 0.05 0.8"/>
+        <box size="0.05 0.7 0.8"/>
       </geometry>
     </collision>
@@ -95,7 +139,7 @@
     <parent link="table_top"/>
     <child link="safety_barrier_back"/>
-    <origin xyz="0.0 0.35 0.75" rpy="0 0 0"/>
+    <origin xyz="-0.15 -0.05 0.75" rpy="0 0 0"/>
   </joint>
-  <!-- Front Barrier -->
+  <!-- Front Barrier (formerly Left Barrier) -->
   <link name="safety_barrier_front">
     <visual>
@@ -108,7 +152,7 @@
     </visual>
     <collision>
-      <origin xyz="0 0 0.4" rpy="0 0 0"/>
+      <origin xyz="0 0 0.4" rpy="0 0 1.5708"/>
       <geometry>
-        <box size="1.2 0.05 0.8"/>
+        <box size="0.05 0.7 0.8"/>
       </geometry>
     </collision>
@@ -117,49 +161,5 @@
     <parent link="table_top"/>
     <child link="safety_barrier_front"/>
-    <origin xyz="0.0 -0.35 0.75" rpy="0 0 0"/>
-  </joint>
-  <!-- Left Barrier -->
-  <link name="safety_barrier_left">
-    <visual>
-      <origin xyz="0 0 0" rpy="0 0 0"/>
-      <geometry>
-        <!-- Scale down from mm to m -->
-        <mesh filename="package://ur_workspace_description/meshes/environment/narrow_safety_barrier.stl" scale="0.001 0.001 0.001"/>
-      </geometry>
-      <material name="workspace_safety_yellow"/>
-    </visual>
-    <collision>
-      <origin xyz="0 0 0.4" rpy="0 0 0"/>
-      <geometry>
-        <box size="0.05 0.7 0.8"/>
-      </geometry>
-    </collision>
-  </link>
-  <joint name="table_to_barrier_left" type="fixed">
-    <parent link="table_top"/>
-    <child link="safety_barrier_left"/>
-    <origin xyz="0.6 0.0 0.75" rpy="0 0 0"/>
-  </joint>
-  <!-- Right Barrier -->
-  <link name="safety_barrier_right">
-    <visual>
-      <origin xyz="0 0 0" rpy="0 0 0"/>
-      <geometry>
-        <!-- Scale down from mm to m -->
-        <mesh filename="package://ur_workspace_description/meshes/environment/narrow_safety_barrier.stl" scale="0.001 0.001 0.001"/>
-      </geometry>
-      <material name="workspace_safety_yellow"/>
-    </visual>
-    <collision>
-      <origin xyz="0 0 0.4" rpy="0 0 0"/>
-      <geometry>
-        <box size="0.05 0.7 0.8"/>
-      </geometry>
-    </collision>
-  </link>
-  <joint name="table_to_barrier_right" type="fixed">
-    <parent link="table_top"/>
-    <child link="safety_barrier_right"/>
-    <origin xyz="-0.6 0.0 0.75" rpy="0 0 0"/>
+    <origin xyz="1.64 -0.05 0.75" rpy="0 0 0"/>
   </joint>
   <!-- Top Barrier -->
@@ -176,5 +176,5 @@
       <origin xyz="0 0 0" rpy="0 0 0"/>
       <geometry>
-        <box size="1.2 0.7 0.01"/>
+        <box size="0.7 1.2 0.01"/>
       </geometry>
     </collision>
@@ -183,5 +183,5 @@
     <parent link="table_top"/>
     <child link="safety_barrier_top"/>
-    <origin xyz="0.0 0.0 1.2" rpy="0 0 0"/>
+    <origin xyz="0 -0.05 1.65" rpy="0 0 0"/>
   </joint>
 </robot>

Commit message: placing robot in environment

File: ur_onrobot_control/urdf/robot_with_environment.urdf.xacro (robot description, xacro)
@@ -48,5 +48,5 @@
         cable_connector="true">
         <!-- Robot positioned on table - adjust as needed -->
-        <origin xyz="0.0 0.0 0.75" rpy="0 0 0"/>
+        <origin xyz="0.8 0.55 0.75" rpy="0 0 0"/>
    </xacro:ur_onrobot>
 </robot>

Commit message: placing robot in environment

File: ur_onrobot_control/urdf/robot_with_environment.urdf.xacro (robot description, xacro)
@@ -48,5 +48,5 @@
         cable_connector="true">
         <!-- Robot positioned on table - adjust as needed -->
-        <origin xyz="0.8 0.55 0.75" rpy="0 0 0"/>
+        <origin xyz="0 0.55 0.75" rpy="0 0 0"/>
    </xacro:ur_onrobot>
 </robot>

Commit message: placing robot in environment

File: ur_onrobot_control/urdf/robot_with_environment.urdf.xacro (robot description, xacro)
@@ -48,5 +48,5 @@
         cable_connector="true">
         <!-- Robot positioned on table - adjust as needed -->
-        <origin xyz="0 0.55 0.75" rpy="0 0 0"/>
+        <origin xyz="0.55 0.8 0.75" rpy="0 0 0"/>
    </xacro:ur_onrobot>
 </robot>

Commit message: placing robot in environment

File: ur_onrobot_control/urdf/robot_with_environment.urdf.xacro (robot description, xacro)
@@ -48,5 +48,5 @@
         cable_connector="true">
         <!-- Robot positioned on table - adjust as needed -->
-        <origin xyz="0.55 0.8 0.75" rpy="0 0 0"/>
+        <origin xyz="0.55 0.65 0.75" rpy="0 0 0"/>
    </xacro:ur_onrobot>
 </robot>
