Commit message: placing robot in environment

File: ur_onrobot_control/urdf/robot_with_right_environment.urdf.xacro (robot description, xacro)
@@ -48,5 +48,5 @@
         cable_connector="true">
         <!-- Robot positioned on table - adjust as needed -->
-        <origin xyz="0.55 0.65 0.75" rpy="0 0 0"/>
+        <origin xyz="0.15 0.65 0.75" rpy="0 0 0"/>
    </xacro:ur_onrobot>
 </robot>
