Commit message: Rotating simulation robot

File: ur_onrobot_control/urdf/right_robot_with_environment.urdf.xacro (robot description, xacro)
@@ -41,5 +41,5 @@
         cable_connector="$(arg cable_connector)">
         <!-- Robot positioned on table - ORIGEN FIJO -->
-        <origin xyz="0.55 0.65 0.75" rpy="0 0 0"/>
+        <origin xyz="0.55 0.65 0.75" rpy="0 0 -1.570796327"/>
    </xacro:ur_onrobot>
 </robot>
