Commit message: environment integration

File: ur_onrobot_control/urdf/left_robot_with_environment.urdf.xacro (robot description, xacro)
@@ -1,4 +1,4 @@
 <?xml version='1.0' encoding='utf-8'?>
-<robot xmlns:xacro="http://www.ros.org/wiki/xacro" name="ur_onrobot_with_environment">
+<robot xmlns:xacro="http://www.ros.org/wiki/xacro" name="left_robot_with_environment">
    <!-- World Link -->
    <link name="world"/>
@@ -7,8 +7,9 @@
    <!-- Create robot description -->
    <xacro:include filename="$(find ur_onrobot_description)/urdf/ur_onrobot_macro.xacro"/>
+   <!-- Define parameters with defaults -->
    <xacro:arg name="ur_type" default="ur5e"/>
    <xacro:arg name="onrobot_type" default="2fg7"/>
-   <xacro:arg name="robot_ip" default="192.168.1.101" />
-   <xacro:arg name="use_fake_hardware" default="true" />
+   <xacro:arg name="robot_ip" default="192.168.1.105"/>
+   <xacro:arg name="use_fake_hardware" default="true"/>
    <xacro:arg name="tf_prefix" default=""/>
    <!-- MODBUS parameters for gripper -->
@@ -17,14 +18,7 @@
    <xacro:arg name="port" default="502"/>
    <xacro:arg name="device_address" default="65"/>
-   <xacro:arg name="device" default="/tmp/ttyUR"/>
-   <!-- Joint limits and other UR parameters -->
-   <xacro:arg name="joint_limits_parameters_file" default="$(find ur_description)/config/$(arg ur_type)/joint_limits.yaml"/>
-   <xacro:arg name="kinematics_parameters_file" default="$(find ur_description)/config/$(arg ur_type)/default_kinematics.yaml"/>
-   <xacro:arg name="physical_parameters_file" default="$(find ur_description)/config/$(arg ur_type)/physical_parameters.yaml"/>
-   <xacro:arg name="visual_parameters_file" default="$(find ur_description)/config/$(arg ur_type)/visual_parameters.yaml"/>
-   <xacro:arg name="script_filename" default="$(find ur_robot_driver)/resources/ros_control.urscript"/>
-   <xacro:arg name="output_recipe_filename" default="$(find ur_robot_driver)/resources/rtde_output_recipe.txt"/>
-   <xacro:arg name="input_recipe_filename" default="$(find ur_robot_driver)/resources/rtde_input_recipe.txt"/>
-   <!-- MAIN ROBOT - Attached to the first table in the environment -->
+   <!-- Cable connector (visual elements) -->
+   <xacro:arg name="cable_connector" default="true"/>
+   <!-- MAIN ROBOT - Attached to table_top in environment -->
    <xacro:ur_onrobot
         parent="table_top"
@@ -34,18 +28,17 @@
         tf_prefix="$(arg tf_prefix)"
         use_fake_hardware="$(arg use_fake_hardware)"
-        joint_limits_parameters_file="$(arg joint_limits_parameters_file)"
-        kinematics_parameters_file="$(arg kinematics_parameters_file)"
-        physical_parameters_file="$(arg physical_parameters_file)"
-        visual_parameters_file="$(arg visual_parameters_file)"
-        script_filename="$(arg script_filename)"
-        output_recipe_filename="$(arg output_recipe_filename)"
-        input_recipe_filename="$(arg input_recipe_filename)"
+        joint_limits_parameters_file="$(find ur_description)/config/$(arg ur_type)/joint_limits.yaml"
+        kinematics_parameters_file="$(find ur_description)/config/$(arg ur_type)/default_kinematics.yaml"
+        physical_parameters_file="$(find ur_description)/config/$(arg ur_type)/physical_parameters.yaml"
+        visual_parameters_file="$(find ur_description)/config/$(arg ur_type)/visual_parameters.yaml"
+        script_filename="$(find ur_robot_driver)/resources/ros_control.urscript"
+        output_recipe_filename="$(find ur_robot_driver)/resources/rtde_output_recipe.txt"
+        input_recipe_filename="$(find ur_robot_driver)/resources/rtde_input_recipe.txt"
         connection_type="$(arg connection_type)"
         ip_address="$(arg ip_address)"
         port="$(arg port)"
         device_address="$(arg device_address)"
-        device="$(arg device)"
-        cable_connector="true">
-        <!-- Robot positioned on table - adjust as needed -->
+        cable_connector="$(arg cable_connector)">
+        <!-- Robot positioned on table - ORIGEN FIJO -->
         <origin xyz="0.15 0.65 0.75" rpy="0 0 0"/>
    </xacro:ur_onrobot>

File: ur_onrobot_control/urdf/right_robot_with_environment.urdf.xacro (robot description, xacro)
@@ -1,4 +1,4 @@
 <?xml version='1.0' encoding='utf-8'?>
-<robot xmlns:xacro="http://www.ros.org/wiki/xacro" name="ur_onrobot_with_environment">
+<robot xmlns:xacro="http://www.ros.org/wiki/xacro" name="right_robot_with_environment">
    <!-- World Link -->
    <link name="world"/>
@@ -7,8 +7,9 @@
    <!-- Create robot description -->
    <xacro:include filename="$(find ur_onrobot_description)/urdf/ur_onrobot_macro.xacro"/>
+   <!-- Define parameters with defaults -->
    <xacro:arg name="ur_type" default="ur5e"/>
    <xacro:arg name="onrobot_type" default="2fg7"/>
-   <xacro:arg name="robot_ip" default="192.168.1.101" />
-   <xacro:arg name="use_fake_hardware" default="true" />
+   <xacro:arg name="robot_ip" default="192.168.1.101"/>
+   <xacro:arg name="use_fake_hardware" default="true"/>
    <xacro:arg name="tf_prefix" default=""/>
    <!-- MODBUS parameters for gripper -->
@@ -17,14 +18,7 @@
    <xacro:arg name="port" default="502"/>
    <xacro:arg name="device_address" default="65"/>
-   <xacro:arg name="device" default="/tmp/ttyUR"/>
-   <!-- Joint limits and other UR parameters -->
-   <xacro:arg name="joint_limits_parameters_file" default="$(find ur_description)/config/$(arg ur_type)/joint_limits.yaml"/>
-   <xacro:arg name="kinematics_parameters_file" default="$(find ur_description)/config/$(arg ur_type)/default_kinematics.yaml"/>
-   <xacro:arg name="physical_parameters_file" default="$(find ur_description)/config/$(arg ur_type)/physical_parameters.yaml"/>
-   <xacro:arg name="visual_parameters_file" default="$(find ur_description)/config/$(arg ur_type)/visual_parameters.yaml"/>
-   <xacro:arg name="script_filename" default="$(find ur_robot_driver)/resources/ros_control.urscript"/>
-   <xacro:arg name="output_recipe_filename" default="$(find ur_robot_driver)/resources/rtde_output_recipe.txt"/>
-   <xacro:arg name="input_recipe_filename" default="$(find ur_robot_driver)/resources/rtde_input_recipe.txt"/>
-   <!-- MAIN ROBOT - Attached to the first table in the environment -->
+   <!-- Cable connector (visual elements) -->
+   <xacro:arg name="cable_connector" default="true"/>
+   <!-- MAIN ROBOT - Attached to table_top in environment -->
    <xacro:ur_onrobot
         parent="table_top"
@@ -34,18 +28,17 @@
         tf_prefix="$(arg tf_prefix)"
         use_fake_hardware="$(arg use_fake_hardware)"
-        joint_limits_parameters_file="$(arg joint_limits_parameters_file)"
-        kinematics_parameters_file="$(arg kinematics_parameters_file)"
-        physical_parameters_file="$(arg physical_parameters_file)"
-        visual_parameters_file="$(arg visual_parameters_file)"
-        script_filename="$(arg script_filename)"
-        output_recipe_filename="$(arg output_recipe_filename)"
-        input_recipe_filename="$(arg input_recipe_filename)"
+        joint_limits_parameters_file="$(find ur_description)/config/$(arg ur_type)/joint_limits.yaml"
+        kinematics_parameters_file="$(find ur_description)/config/$(arg ur_type)/default_kinematics.yaml"
+        physical_parameters_file="$(find ur_description)/config/$(arg ur_type)/physical_parameters.yaml"
+        visual_parameters_file="$(find ur_description)/config/$(arg ur_type)/visual_parameters.yaml"
+        script_filename="$(find ur_robot_driver)/resources/ros_control.urscript"
+        output_recipe_filename="$(find ur_robot_driver)/resources/rtde_output_recipe.txt"
+        input_recipe_filename="$(find ur_robot_driver)/resources/rtde_input_recipe.txt"
         connection_type="$(arg connection_type)"
         ip_address="$(arg ip_address)"
         port="$(arg port)"
         device_address="$(arg device_address)"
-        device="$(arg device)"
-        cable_connector="true">
-        <!-- Robot positioned on table - adjust as needed -->
+        cable_connector="$(arg cable_connector)">
+        <!-- Robot positioned on table - ORIGEN FIJO -->
         <origin xyz="0.55 0.65 0.75" rpy="0 0 0"/>
    </xacro:ur_onrobot>

File: ur_onrobot_description/urdf/ur_onrobot.urdf.xacro (robot description, xacro)
@@ -42,5 +42,5 @@
         device_address="$(arg device_address)"
         >
-        <origin xyz="0 0 1" rpy="0 0 0" />
+        <origin xyz="0 0 0" rpy="0 0 0" />
     </xacro:ur_onrobot>
 </robot>

Commit message: Rotating left simulation robot - fix

File: ur_onrobot_control/urdf/left_robot_with_environment.urdf.xacro (robot description, xacro)
@@ -41,5 +41,5 @@
         cable_connector="$(arg cable_connector)">
         <!-- Robot positioned on table - ORIGEN FIJO -->
-        <origin xyz="0.15 0.65 0.75" rpy="0 0 0"/>
+        <origin xyz="0.15 0.65 0.75" rpy="0 0 1.570796327"/>
    </xacro:ur_onrobot>
 </robot>
