Commit message: Robot Base locked at (0,0,0,0,0,0)

File: ur_onrobot_control/urdf/left_robot_with_environment.urdf.xacro (robot description, xacro)
@@ -20,7 +20,7 @@
    <!-- Cable connector (visual elements) -->
    <xacro:arg name="cable_connector" default="true"/>
-   <!-- MAIN ROBOT - Attached to table_top in environment -->
+   <!-- MAIN ROBOT - Attached to world at origin (0,0,0) -->
    <xacro:ur_onrobot
-        parent="table_top"
+        parent="world"
         robot_ip="$(arg robot_ip)"
         ur_type="$(arg ur_type)"
@@ -40,6 +40,6 @@
         device_address="$(arg device_address)"
         cable_connector="$(arg cable_connector)">
-        <!-- Robot positioned on table - ORIGEN FIJO -->
-        <origin xyz="0.15 0.65 0.75" rpy="0 0 1.570796327"/>
+        <!-- Robot base at world origin (0,0,0) -->
+        <origin xyz="0 0 0" rpy="0 0 1.570796327"/>
    </xacro:ur_onrobot>
 </robot>

File: ur_onrobot_control/urdf/right_robot_with_environment.urdf.xacro (robot description, xacro)
@@ -20,7 +20,7 @@
    <!-- Cable connector (visual elements) -->
    <xacro:arg name="cable_connector" default="true"/>
-   <!-- MAIN ROBOT - Attached to table_top in environment -->
+   <!-- MAIN ROBOT - Attached to world at origin (0,0,0) -->
    <xacro:ur_onrobot
-        parent="table_top"
+        parent="world"
         robot_ip="$(arg robot_ip)"
         ur_type="$(arg ur_type)"
@@ -40,6 +40,6 @@
         device_address="$(arg device_address)"
         cable_connector="$(arg cable_connector)">
-        <!-- Robot positioned on table - ORIGEN FIJO -->
-        <origin xyz="0.55 0.65 0.75" rpy="0 0 -1.570796327"/>
+        <!-- Robot base at world origin (0,0,0) -->
+        <origin xyz="0 0 0" rpy="0 0 -1.570796327"/>
    </xacro:ur_onrobot>
 </robot>

File: ur_workspace_description/urdf/Only_environment_for_left_robot.urdf.xacro (robot description, xacro)
@@ -26,5 +26,5 @@
     <child link="table_top"/>
     <!-- Rotated 90 degrees around Z-axis like in reference file -->
-    <origin xyz="0 0.05 0" rpy="0 0 0"/>
+    <origin xyz="-0.15 -0.65 -0.75" rpy="0 0 0"/>
   </joint>
   <!-- Conveyor Belt -->
@@ -49,5 +49,5 @@
     <child link="conveyor_belt"/>
     <!-- Conveyor rotated 90 degrees and positioned between tables -->
-    <origin xyz="-0.87 0 0" rpy="0 0 0"/>
+    <origin xyz="-1.02 -0.70 -0.75" rpy="0 0 0"/>
   </joint>
   <!-- Second Table -->
@@ -72,5 +72,5 @@
     <child link="table_top_2"/>
     <!-- Second table positioned on the other side of conveyor with 90-degree rotation -->
-    <origin xyz="-1.64 0.05 0" rpy="0 0 0"/>
+    <origin xyz="-1.79 -0.65 -0.75" rpy="0 0 0"/>
   </joint>
   <!-- Safety Barriers - Adjusted positions for 90-degree rotated tables -->

File: ur_workspace_description/urdf/Only_environment_for_right_robot.urdf.xacro (robot description, xacro)
@@ -26,5 +26,5 @@
     <child link="table_top"/>
     <!-- Rotated 90 degrees around Z-axis like in reference file -->
-    <origin xyz="0 0.05 0" rpy="0 0 0"/>
+    <origin xyz="-0.55 -0.65 -0.75" rpy="0 0 0"/>
   </joint>
   <!-- Conveyor Belt -->
@@ -49,5 +49,5 @@
     <child link="conveyor_belt"/>
     <!-- Conveyor rotated 90 degrees and positioned between tables -->
-    <origin xyz="0.77 0 0" rpy="0 0 0"/>
+    <origin xyz="0.22 -0.70 -0.75" rpy="0 0 0"/>
   </joint>
   <!-- Second Table -->
@@ -72,5 +72,5 @@
     <child link="table_top_2"/>
     <!-- Second table positioned on the other side of conveyor with 90-degree rotation -->
-    <origin xyz="1.64 0.05 0" rpy="0 0 0"/>
+    <origin xyz="1.09 -0.65 -0.75" rpy="0 0 0"/>
   </joint>
   <!-- Safety Barriers - Adjusted positions for 90-degree rotated tables -->

File: ur_workspace_description/urdf/left_robot_environment.urdf.xacro (robot description, xacro)
@@ -24,5 +24,5 @@
     <child link="table_top"/>
     <!-- Rotated 90 degrees around Z-axis like in reference file -->
-    <origin xyz="0 0.05 0" rpy="0 0 0"/>
+    <origin xyz="-0.15 -0.65 -0.75" rpy="0 0 0"/>
   </joint>
   <!-- Conveyor Belt -->
@@ -47,5 +47,5 @@
     <child link="conveyor_belt"/>
     <!-- Conveyor rotated 90 degrees and positioned between tables -->
-    <origin xyz="-0.87 0 0" rpy="0 0 0"/>
+    <origin xyz="-1.02 -0.70 -0.75" rpy="0 0 0"/>
   </joint>
   <!-- Second Table -->
@@ -70,5 +70,5 @@
     <child link="table_top_2"/>
     <!-- Second table positioned on the other side of conveyor with 90-degree rotation -->
-    <origin xyz="-1.64 0.05 0" rpy="0 0 0"/>
+    <origin xyz="-1.79 -0.65 -0.75" rpy="0 0 0"/>
   </joint>
   <!-- Safety Barriers - Adjusted positions for 90-degree rotated tables -->

File: ur_workspace_description/urdf/right_robot_environment.urdf.xacro (robot description, xacro)
@@ -24,5 +24,5 @@
     <child link="table_top"/>
     <!-- Rotated 90 degrees around Z-axis like in reference file -->
-    <origin xyz="0 0.05 0" rpy="0 0 0"/>
+    <origin xyz="-0.55 -0.65 -0.75" rpy="0 0 0"/>
   </joint>
   <!-- Conveyor Belt -->
@@ -47,5 +47,5 @@
     <child link="conveyor_belt"/>
     <!-- Conveyor rotated 90 degrees and positioned between tables -->
-    <origin xyz="0.77 0 0" rpy="0 0 0"/>
+    <origin xyz="0.22 -0.70 -0.75" rpy="0 0 0"/>
   </joint>
   <!-- Second Table -->
@@ -70,5 +70,5 @@
     <child link="table_top_2"/>
     <!-- Second table positioned on the other side of conveyor with 90-degree rotation -->
-    <origin xyz="1.64 0.05 0" rpy="0 0 0"/>
+    <origin xyz="1.09 -0.65 -0.75" rpy="0 0 0"/>
   </joint>
   <!-- Safety Barriers - Adjusted positions for 90-degree rotated tables -->
