Commit message: OnRobot 2FG7 addition - Inclusion package 1

File: ur_onrobot_moveit_config/srdf/ur_onrobot.srdf.xacro (robot description, xacro)
@@ -5,5 +5,16 @@
   <!-- parameters -->
   <xacro:arg name="prefix" default="" />
+  <xacro:arg name="onrobot_type" default="rg2" />
   <xacro:include filename="$(find ur_onrobot_moveit_config)/srdf/ur_onrobot_macro.srdf.xacro"/>
+  <xacro:include filename="$(find ur_onrobot_moveit_config)/srdf/ur_onrobot_rg.srdf.xacro"/>
+  <xacro:include filename="$(find ur_onrobot_moveit_config)/srdf/ur_onrobot_2fg7.srdf.xacro"/>
+  <!-- Common robot configuration -->
   <xacro:ur_onrobot_srdf name="$(arg name)" prefix="$(arg prefix)"/>
+  <!-- Gripper-specific configuration -->
+  <xacro:if value="$(arg onrobot_type) == 'rg2' or $(arg onrobot_type) == 'rg6'">
+    <xacro:ur_onrobot_rg_srdf name="$(arg name)" prefix="$(arg prefix)"/>
+  </xacro:if>
+  <xacro:if value="$(arg onrobot_type) == '2fg7' or $(arg onrobot_type) == '2fg14'">
+    <xacro:ur_onrobot_2fg7_srdf name="$(arg name)" prefix="$(arg prefix)"/>
+  </xacro:if>
 </robot>

File: ur_onrobot_moveit_config/srdf/ur_onrobot_macro.srdf.xacro (robot description, xacro)
@@ -1,39 +1,11 @@
 <?xml version="1.0" encoding="UTF-8"?>
 <robot xmlns:xacro="http://wiki.ros.org/xacro">
-<!--This does not replace URDF, and is not an extension of URDF.
-    This is a format for representing semantic information about the robot structure.
-    A URDF file must exist for this robot as well, where the joints and the links that are referenced are defined
--->
   <xacro:macro name="ur_onrobot_srdf" params="name prefix">
     <!--GROUPS - Representation of a set of joints and links. This can be useful for specifying DOF to plan for, defining arms, end effectors, etc-->
-    <!--LINKS - When a link is specified, the parent joint of that link (if it exists) is automatically included-->
-    <!--JOINTS - When a joint is specified, the child link of that joint (which will always exist) is automatically included-->
-    <!--CHAINS - When a chain is specified, all the links along the chain (including endpoints) are included in the group. Additionally, all the joints that are parents to included links are also included. This means that joints along the chain and the parent joint of the base link are included in the group-->
-    <!--SUBGROUPS - Groups can also be formed by referencing to already defined group names-->
-    <group name="${prefix}${name}_gripper">
-      <link name="${prefix}onrobot_base_link"/>
-      <link name="${prefix}cable_connector_0"/>
-      <link name="${prefix}cable_connector_1"/>
-      <link name="${prefix}left_inner_knuckle"/>
-      <link name="${prefix}left_outer_knuckle"/>
-      <link name="${prefix}left_inner_finger"/>
-      <link name="${prefix}left_finger_tip"/>
-      <link name="${prefix}right_inner_knuckle"/>
-      <link name="${prefix}right_outer_knuckle"/>
-      <link name="${prefix}right_inner_finger"/>
-      <link name="${prefix}right_finger_tip"/>
-      <link name="${prefix}finger_width_mock_link"/>
-      <link name="${prefix}gripper_tcp"/>
-    </group>
+    <!-- COMMON GROUPS FOR ALL GRIPPERS -->
     <group name="${prefix}${name}_manipulator">
       <chain base_link="${prefix}base_link" tip_link="${prefix}gripper_tcp" />
     </group>
-    <!--GROUP STATES - Purpose - Define a named state for a particular group, in terms of joint values. This is useful to define states like 'folded arms'-->
-    <group_state name="closed" group="${prefix}${name}_gripper">
-      <joint name="finger_width" value="0.0"/>
-    </group_state>
-    <group_state name="open" group="${prefix}${name}_gripper">
-      <joint name="finger_width" value="0.100"/>
-    </group_state>
+    <!-- COMMON ROBOT STATES -->
     <group_state name="${prefix}home" group="${prefix}${name}_manipulator">
       <joint name="${prefix}elbow_joint" value="0" />
@@ -62,6 +34,5 @@
     <!--END EFFECTOR - Purpose - Represent information about an end effector.-->
     <end_effector name="${prefix}${name}_tcp" parent_link="${prefix}gripper_tcp" group="${prefix}${name}_gripper" parent_group="${prefix}${name}_manipulator"/>
-    <!--VIRTUAL JOINT - Purpose - this element defines a virtual joint between a robot link and an external frame of reference (considered fixed with respect to the robot)-->
-    <!--DISABLE COLLISIONS - By default it is assumed that any link of the robot could potentially come into collision with any other link in the robot. This tag disables collision checking between a specified pair of links. -->
+    <!-- COMMON COLLISION DISABLEMENTS (robot arm only) -->
     <disable_collisions link1="${prefix}base_link" link2="${prefix}base_link_inertia" reason="Adjacent" />
     <disable_collisions link1="${prefix}base_link_inertia" link2="${prefix}shoulder_link" reason="Adjacent" />
@@ -75,67 +46,18 @@
     <disable_collisions link1="${prefix}wrist_1_link" link2="${prefix}wrist_3_link" reason="Never" />
     <disable_collisions link1="${prefix}wrist_2_link" link2="${prefix}wrist_3_link" reason="Adjacent" />
+    <!-- COMMON GRIPPER COLLISIONS (cable connectors) -->
     <disable_collisions link1="${prefix}cable_connector_0" link2="${prefix}cable_connector_1" reason="Never"/>
-    <disable_collisions link1="${prefix}cable_connector_0" link2="${prefix}left_inner_finger" reason="Never"/>
-    <disable_collisions link1="${prefix}cable_connector_0" link2="${prefix}left_inner_knuckle" reason="Never"/>
-    <disable_collisions link1="${prefix}cable_connector_0" link2="${prefix}left_outer_knuckle" reason="Never"/>
     <disable_collisions link1="${prefix}cable_connector_0" link2="${prefix}onrobot_base_link" reason="Adjacent"/>
-    <disable_collisions link1="${prefix}cable_connector_0" link2="${prefix}right_inner_finger" reason="Never"/>
-    <disable_collisions link1="${prefix}cable_connector_0" link2="${prefix}right_inner_knuckle" reason="Never"/>
-    <disable_collisions link1="${prefix}cable_connector_0" link2="${prefix}right_outer_knuckle" reason="Never"/>
+    <disable_collisions link1="${prefix}cable_connector_1" link2="${prefix}onrobot_base_link" reason="Adjacent"/>
     <disable_collisions link1="${prefix}cable_connector_0" link2="${prefix}wrist_1_link" reason="Never"/>
     <disable_collisions link1="${prefix}cable_connector_0" link2="${prefix}wrist_2_link" reason="Never"/>
     <disable_collisions link1="${prefix}cable_connector_0" link2="${prefix}wrist_3_link" reason="Default"/>
-    <disable_collisions link1="${prefix}cable_connector_1" link2="${prefix}left_inner_finger" reason="Never"/>
-    <disable_collisions link1="${prefix}cable_connector_1" link2="${prefix}left_inner_knuckle" reason="Never"/>
-    <disable_collisions link1="${prefix}cable_connector_1" link2="${prefix}left_outer_knuckle" reason="Never"/>
-    <disable_collisions link1="${prefix}cable_connector_1" link2="${prefix}onrobot_base_link" reason="Adjacent"/>
-    <disable_collisions link1="${prefix}cable_connector_1" link2="${prefix}right_inner_finger" reason="Never"/>
-    <disable_collisions link1="${prefix}cable_connector_1" link2="${prefix}right_inner_knuckle" reason="Never"/>
-    <disable_collisions link1="${prefix}cable_connector_1" link2="${prefix}right_outer_knuckle" reason="Never"/>
     <disable_collisions link1="${prefix}cable_connector_1" link2="${prefix}wrist_1_link" reason="Never"/>
     <disable_collisions link1="${prefix}cable_connector_1" link2="${prefix}wrist_2_link" reason="Default"/>
     <disable_collisions link1="${prefix}cable_connector_1" link2="${prefix}wrist_3_link" reason="Default"/>
-    <disable_collisions link1="${prefix}left_inner_finger" link2="${prefix}left_inner_knuckle" reason="Default"/>
-    <disable_collisions link1="${prefix}left_inner_finger" link2="${prefix}left_outer_knuckle" reason="Adjacent"/>
-    <disable_collisions link1="${prefix}left_inner_finger" link2="${prefix}onrobot_base_link" reason="Never"/>
-    <disable_collisions link1="${prefix}left_inner_finger" link2="${prefix}right_inner_finger" reason="Default"/>
-    <disable_collisions link1="${prefix}left_inner_finger" link2="${prefix}right_inner_knuckle" reason="Never"/>
-    <disable_collisions link1="${prefix}left_inner_finger" link2="${prefix}right_outer_knuckle" reason="Never"/>
-    <disable_collisions link1="${prefix}left_inner_finger" link2="${prefix}wrist_1_link" reason="Never"/>
-    <disable_collisions link1="${prefix}left_inner_finger" link2="${prefix}wrist_2_link" reason="Never"/>
-    <disable_collisions link1="${prefix}left_inner_finger" link2="${prefix}wrist_3_link" reason="Never"/>
-    <disable_collisions link1="${prefix}left_inner_knuckle" link2="${prefix}left_outer_knuckle" reason="Default"/>
-    <disable_collisions link1="${prefix}left_inner_knuckle" link2="${prefix}onrobot_base_link" reason="Adjacent"/>
-    <disable_collisions link1="${prefix}left_inner_knuckle" link2="${prefix}right_inner_finger" reason="Never"/>
-    <disable_collisions link1="${prefix}left_inner_knuckle" link2="${prefix}right_inner_knuckle" reason="Never"/>
-    <disable_collisions link1="${prefix}left_inner_knuckle" link2="${prefix}right_outer_knuckle" reason="Never"/>
-    <disable_collisions link1="${prefix}left_inner_knuckle" link2="${prefix}wrist_1_link" reason="Never"/>
-    <disable_collisions link1="${prefix}left_inner_knuckle" link2="${prefix}wrist_2_link" reason="Never"/>
-    <disable_collisions link1="${prefix}left_inner_knuckle" link2="${prefix}wrist_3_link" reason="Never"/>
-    <disable_collisions link1="${prefix}left_outer_knuckle" link2="${prefix}onrobot_base_link" reason="Adjacent"/>
-    <disable_collisions link1="${prefix}left_outer_knuckle" link2="${prefix}right_inner_finger" reason="Never"/>
-    <disable_collisions link1="${prefix}left_outer_knuckle" link2="${prefix}right_inner_knuckle" reason="Never"/>
-    <disable_collisions link1="${prefix}left_outer_knuckle" link2="${prefix}right_outer_knuckle" reason="Never"/>
-    <disable_collisions link1="${prefix}left_outer_knuckle" link2="${prefix}wrist_1_link" reason="Never"/>
-    <disable_collisions link1="${prefix}left_outer_knuckle" link2="${prefix}wrist_2_link" reason="Never"/>
-    <disable_collisions link1="${prefix}left_outer_knuckle" link2="${prefix}wrist_3_link" reason="Never"/>
-    <disable_collisions link1="${prefix}onrobot_base_link" link2="${prefix}right_inner_finger" reason="Never"/>
-    <disable_collisions link1="${prefix}onrobot_base_link" link2="${prefix}right_inner_knuckle" reason="Adjacent"/>
-    <disable_collisions link1="${prefix}onrobot_base_link" link2="${prefix}right_outer_knuckle" reason="Adjacent"/>
+    <!-- COMMON GRIPPER TO ROBOT COLLISIONS -->
     <disable_collisions link1="${prefix}onrobot_base_link" link2="${prefix}wrist_1_link" reason="Never"/>
     <disable_collisions link1="${prefix}onrobot_base_link" link2="${prefix}wrist_2_link" reason="Never"/>
     <disable_collisions link1="${prefix}onrobot_base_link" link2="${prefix}wrist_3_link" reason="Adjacent"/>
-    <disable_collisions link1="${prefix}right_inner_finger" link2="${prefix}right_inner_knuckle" reason="Default"/>
-    <disable_collisions link1="${prefix}right_inner_finger" link2="${prefix}right_outer_knuckle" reason="Adjacent"/>
-    <disable_collisions link1="${prefix}right_inner_finger" link2="${prefix}wrist_1_link" reason="Never"/>
-    <disable_collisions link1="${prefix}right_inner_finger" link2="${prefix}wrist_2_link" reason="Never"/>
-    <disable_collisions link1="${prefix}right_inner_finger" link2="${prefix}wrist_3_link" reason="Never"/>
-    <disable_collisions link1="${prefix}right_inner_knuckle" link2="${prefix}right_outer_knuckle" reason="Default"/>
-    <disable_collisions link1="${prefix}right_inner_knuckle" link2="${prefix}wrist_1_link" reason="Never"/>
-    <disable_collisions link1="${prefix}right_inner_knuckle" link2="${prefix}wrist_2_link" reason="Never"/>
-    <disable_collisions link1="${prefix}right_inner_knuckle" link2="${prefix}wrist_3_link" reason="Never"/>
-    <disable_collisions link1="${prefix}right_outer_knuckle" link2="${prefix}wrist_1_link" reason="Never"/>
-    <disable_collisions link1="${prefix}right_outer_knuckle" link2="${prefix}wrist_2_link" reason="Never"/>
-    <disable_collisions link1="${prefix}right_outer_knuckle" link2="${prefix}wrist_3_link" reason="Never"/>
   </xacro:macro>
 </robot>

Commit message: moveit package fix

File: ur_onrobot_moveit_config/srdf/ur_onrobot.srdf.xacro (robot description, xacro)
@@ -1,7 +1,5 @@
 <?xml version="1.0" encoding="UTF-8"?>
 <robot xmlns:xacro="http://wiki.ros.org/xacro" name="$(arg name)">
-  <!-- robot name parameter -->
   <xacro:arg name="name" default="ur_onrobot"/>
-  <!-- parameters -->
   <xacro:arg name="prefix" default="" />
   <xacro:arg name="onrobot_type" default="rg2" />
@@ -12,8 +10,9 @@
   <xacro:ur_onrobot_srdf name="$(arg name)" prefix="$(arg prefix)"/>
   <!-- Gripper-specific configuration -->
-  <xacro:if value="${onrobot_type in ['rg2', 'rg6']}">
+  <xacro:property name="gripper" value="$(arg onrobot_type)" />
+  <xacro:if value="${gripper == 'rg2' or gripper == 'rg6'}">
     <xacro:ur_onrobot_rg_srdf name="$(arg name)" prefix="$(arg prefix)"/>
   </xacro:if>
-  <xacro:if value="${onrobot_type in ['2fg7', '2fg14']}">
+  <xacro:if value="${gripper == '2fg7' or gripper == '2fg14'}">
     <xacro:ur_onrobot_2fg7_srdf name="$(arg name)" prefix="$(arg prefix)"/>
   </xacro:if>

Commit message: moveit package fix - 1

File: ur_onrobot_moveit_config/srdf/ur_onrobot.srdf.xacro (robot description, xacro)
@@ -1,7 +1,5 @@
 <?xml version="1.0" encoding="UTF-8"?>
 <robot xmlns:xacro="http://wiki.ros.org/xacro" name="$(arg name)">
-  <!-- robot name parameter -->
   <xacro:arg name="name" default="ur_onrobot"/>
-  <!-- parameters -->
   <xacro:arg name="prefix" default="" />
   <xacro:arg name="onrobot_type" default="rg2" />
@@ -12,8 +10,9 @@
   <xacro:ur_onrobot_srdf name="$(arg name)" prefix="$(arg prefix)"/>
   <!-- Gripper-specific configuration -->
-  <xacro:if value="${onrobot_type == 'rg2' or onrobot_type == 'rg6'}">
+  <xacro:property name="gripper" value="$(arg onrobot_type)" />
+  <xacro:if value="${gripper == 'rg2' or gripper == 'rg6'}">
     <xacro:ur_onrobot_rg_srdf name="$(arg name)" prefix="$(arg prefix)"/>
   </xacro:if>
-  <xacro:if value="${onrobot_type == '2fg7' or onrobot_type == '2fg14'}">
+  <xacro:if value="${gripper == '2fg7' or gripper == '2fg14'}">
     <xacro:ur_onrobot_2fg7_srdf name="$(arg name)" prefix="$(arg prefix)"/>
   </xacro:if>
