Commit message: Refactor launch files for unified robot configuration and enhance environment support

File: ur_onrobot_moveit_config/srdf/ur_onrobot.srdf.xacro (robot description, xacro)
@@ -1,5 +1,6 @@
 <?xml version="1.0" encoding="utf-8"?>
-<robot xmlns:xacro="http://www.ros.org/wiki/xacro" name="ur_onrobot">
+<robot xmlns:xacro="http://www.ros.org/wiki/xacro" name="$(arg robot_name)">
   <!-- Arguments for dynamic resolution -->
+  <xacro:arg name="robot_name" default="ur_onrobot"/>
   <xacro:arg name="onrobot_type" default="2fg7"/>
   <xacro:arg name="sim_env" default="basic"/>

File: ur_workspace_description/urdf/Only_environment_for_left_robot.urdf.xacro (robot description, xacro)
@@ -18,5 +18,5 @@
       <origin xyz="0 0 0" rpy="0 0 0"/>
       <geometry>
-        <box size="-1.2 0.7 0.75"/>
+        <box size="1.2 0.7 0.75"/>
       </geometry>
     </collision>
@@ -41,5 +41,5 @@
       <origin xyz="0 0 0" rpy="0 0 0"/>
       <geometry>
-        <box size="-2.05 0.825 0"/>
+        <box size="2.05 0.825 0.05"/>
       </geometry>
     </collision>
@@ -64,5 +64,5 @@
       <origin xyz="0 0 0" rpy="0 0 0"/>
       <geometry>
-        <box size="-1.2 0.7 0.75"/>
+        <box size="1.2 0.7 0.75"/>
       </geometry>
     </collision>
@@ -88,5 +88,5 @@
       <origin xyz="0 0 0.4" rpy="0 0 1.5708"/>
       <geometry>
-        <box size="-1.2 0.05 0.8"/>
+        <box size="1.2 0.05 0.8"/>
       </geometry>
     </collision>
@@ -110,5 +110,5 @@
       <origin xyz="0 0 0.4" rpy="0 0 1.5708"/>
       <geometry>
-        <box size="-1.2 0.05 0.8"/>
+        <box size="1.2 0.05 0.8"/>
       </geometry>
     </collision>
@@ -176,5 +176,5 @@
       <origin xyz="0 0 0" rpy="0 0 0"/>
       <geometry>
-        <box size="-0.7 1.2 0.01"/>
+        <box size="0.7 1.2 0.01"/>
       </geometry>
     </collision>

File: ur_workspace_description/urdf/Only_environment_for_right_robot.urdf.xacro (robot description, xacro)
@@ -41,5 +41,5 @@
       <origin xyz="0 0 0" rpy="0 0 0"/>
       <geometry>
-        <box size="2.05 0.825 0"/>
+        <box size="2.05 0.825 0.05"/>
       </geometry>
     </collision>

File: ur_workspace_description/urdf/left_robot_environment.urdf.xacro (robot description, xacro)
@@ -16,5 +16,5 @@
       <origin xyz="0 0 0" rpy="0 0 0"/>
       <geometry>
-        <box size="-1.2 0.7 0.75"/>
+        <box size="1.2 0.7 0.75"/>
       </geometry>
     </collision>
@@ -39,5 +39,5 @@
       <origin xyz="0 0 0" rpy="0 0 0"/>
       <geometry>
-        <box size="-2.05 0.825 0"/>
+        <box size="2.05 0.825 0.05"/>
       </geometry>
     </collision>
@@ -62,5 +62,5 @@
       <origin xyz="0 0 0" rpy="0 0 0"/>
       <geometry>
-        <box size="-1.2 0.7 0.75"/>
+        <box size="1.2 0.7 0.75"/>
       </geometry>
     </collision>
@@ -86,5 +86,5 @@
       <origin xyz="0 0 0.4" rpy="0 0 1.5708"/>
       <geometry>
-        <box size="-1.2 0.05 0.8"/>
+        <box size="1.2 0.05 0.8"/>
       </geometry>
     </collision>
@@ -108,5 +108,5 @@
       <origin xyz="0 0 0.4" rpy="0 0 1.5708"/>
       <geometry>
-        <box size="-1.2 0.05 0.8"/>
+        <box size="1.2 0.05 0.8"/>
       </geometry>
     </collision>
@@ -174,5 +174,5 @@
       <origin xyz="0 0 0" rpy="0 0 0"/>
       <geometry>
-        <box size="-0.7 1.2 0.01"/>
+        <box size="0.7 1.2 0.01"/>
       </geometry>
     </collision>

File: ur_workspace_description/urdf/right_robot_environment.urdf.xacro (robot description, xacro)
@@ -39,5 +39,5 @@
       <origin xyz="0 0 0" rpy="0 0 0"/>
       <geometry>
-        <box size="2.05 0.825 0"/>
+        <box size="2.05 0.825 0.05"/>
       </geometry>
     </collision>

Commit message: fix(moveit): adapt home pose shoulder_pan_joint to right and left environments to avoid collision

File: ur_onrobot_moveit_config/srdf/ur_onrobot.srdf.xacro (robot description, xacro)
@@ -21,6 +21,15 @@
   </group>
   <!-- ==================== GROUP STATES (ARM) ==================== -->
+  <xacro:if value="${sim_env == 'right'}">
+    <xacro:property name="home_shoulder_pan" value="1.5708"/>
+  </xacro:if>
+  <xacro:if value="${sim_env == 'left'}">
+    <xacro:property name="home_shoulder_pan" value="3.1415"/>
+  </xacro:if>
+  <xacro:if value="${sim_env == 'basic'}">
+    <xacro:property name="home_shoulder_pan" value="-1.5708"/>
+  </xacro:if>
   <group_state name="home" group="ur_manipulator">
-    <joint name="${tf_prefix}shoulder_pan_joint" value="-1.5708"/>
+    <joint name="${tf_prefix}shoulder_pan_joint" value="${home_shoulder_pan}"/>
     <joint name="${tf_prefix}shoulder_lift_joint" value="-1.5708"/>
     <joint name="${tf_prefix}elbow_joint" value="1.5708"/>
