Commit message: Implement UR + OnRobot Pick & Place Node with MoveIt Task Constructor
- Added `ur_onrobot_mtc_node.cpp` for handling pick and place tasks using MoveIt Task Constructor.
- Configured parameters for arm and gripper settings, including poses and distances.
- Implemented a service for executing pick and place tasks on demand.
- Introduced automatic execution on startup with a configurable delay.
- Enhanced planning scene setup with collision objects and optional support table.
- Created a comprehensive task pipeline for pick and place operations, including grasping and releasing mechanisms.
- Updated `moveit_controllers.yaml` to switch default controllers based on hardware simulation.
- Modified `ompl_planning.yaml` to include additional planner configurations.
- Adjusted `pilz_industrial_motion_planner_planning.yaml` to set the planning plugin.
- Updated launch files to dynamically configure controllers based on hardware simulation.
- Added a new launch file `ur_onrobot_mtc.launch.py` for launching the MTC node.
- Included RViz configuration for visualizing motion planning tasks.
- Updated package dependencies in `package.xml` to include MoveIt Task Constructor packages.
- Modified SRDF files to reflect changes in gripper states and arm home position.

File: ur_onrobot_moveit_config/srdf/inc/vgc10_macro.srdf.xacro (robot description, xacro)
@@ -12,16 +12,18 @@
     <group_state name="grip" group="gripper">
       <joint name="${tf_prefix}vacuum_channel_a" value="1.0"/>
-      <joint name="${tf_prefix}vacuum_channel_b" value="1.0"/>
     </group_state>
     <group_state name="release" group="gripper">
       <joint name="${tf_prefix}vacuum_channel_a" value="0.0"/>
-      <joint name="${tf_prefix}vacuum_channel_b" value="0.0"/>
+    </group_state>
+    <group_state name="closed" group="gripper">
+      <joint name="${tf_prefix}vacuum_channel_a" value="1.0"/>
+    </group_state>
+    <group_state name="open" group="gripper">
+      <joint name="${tf_prefix}vacuum_channel_a" value="0.0"/>
     </group_state>
     <group_state name="grip_a" group="gripper">
       <joint name="${tf_prefix}vacuum_channel_a" value="1.0"/>
-      <joint name="${tf_prefix}vacuum_channel_b" value="0.0"/>
     </group_state>
     <group_state name="grip_b" group="gripper">
-      <joint name="${tf_prefix}vacuum_channel_a" value="0.0"/>
       <joint name="${tf_prefix}vacuum_channel_b" value="1.0"/>
     </group_state>

File: ur_onrobot_moveit_config/srdf/ur_onrobot.srdf.xacro (robot description, xacro)
@@ -22,5 +22,5 @@
   <!-- ==================== GROUP STATES (ARM) ==================== -->
   <group_state name="home" group="ur_manipulator">
-    <joint name="${tf_prefix}shoulder_pan_joint" value="0.0"/>
+    <joint name="${tf_prefix}shoulder_pan_joint" value="-1.5708"/>
     <joint name="${tf_prefix}shoulder_lift_joint" value="-1.5708"/>
     <joint name="${tf_prefix}elbow_joint" value="1.5708"/>
