Commit message: fix(gripper): adjust gripper open/close positions for 2FG7 configuration

File: ur_onrobot_moveit_config/srdf/inc/2fg7_macro.srdf.xacro (robot description, xacro)
@@ -10,5 +10,5 @@
     <!-- Group States -->
     <group_state name="open" group="gripper">
-      <joint name="${tf_prefix}finger_width" value="0.070"/>
+      <joint name="${tf_prefix}finger_width" value="0.073"/>
     </group_state>
     <group_state name="closed" group="gripper">
